File: Power Supply/Kicad/untitled.kicad_sch (KiCad schematic)
At the start: 4 parts, among them J1 ZenBus, U1 INA3221, U2 INA3221, U3 STM32L476RGTx

Commit message: commit de teste com o git, adicionado sim. Ltspice
Parts:
- J1: footprint (none) -> Connector_PinHeader_2.54mm:PinHeader_2x20_P2.54mm_Vertical
Connections:
- net GND: now also U1.3 (GND), U2.3 (GND), U3.12 (VSSA), U3.18 (VSS), U3.31 (VSS), U3.47 (VSS), U3.63 (VSS)
Other:
- moved on the sheet: U3

Commit message: Mais adição
Conclusão do esquema dos reguladores e [início da] organização do esquema.
Parts:
- renumbered U3 to U1, U1 to U2, U2 to U3
Other:
- removed sheet 3.3V Regulator
- removed sheet 5V Regulator
Changed lines of the file:
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@@
 		(dnp no)
 		(fields_autoplaced yes)
-		(property "Reference" "#PWR01"
+		(property "Reference" "#PWR04"
 			(at 267.97 59.69 0)
 			(hide yes)
@@
 			(project "Power Supply ZensatV3"
 				(path "/6407b9bb-bcf3-46ce-88dc-7e023cbc9b7f"
-					(reference "#PWR01")
+					(reference "#PWR04")
 					(unit 1)
 				)
@@
 		(dnp no)
 		(fields_autoplaced yes)
-		(property "Reference" "U1"
+		(property "Reference" "U2"
 			(at 127.8733 81.28 0)
 			(show_name no)
@@
 			(project "Power Supply ZensatV3"
 				(path "/6407b9bb-bcf3-46ce-88dc-7e023cbc9b7f"
-					(reference "U1")
+					(reference "U2")
 					(unit 1)
 				)
@@
 		(dnp no)
 		(fields_autoplaced yes)
-		(property "Reference" "#PWR04"
+		(property "Reference" "#PWR02"
 			(at 120.65 125.73 0)
 			(hide yes)
@@
 			(project "Power Supply ZensatV3"
 				(path "/6407b9bb-bcf3-46ce-88dc-7e023cbc9b7f"
-					(reference "#PWR04")
+					(reference "#PWR02")
 					(unit 1)
 				)
@@
 		(dnp no)
 		(fields_autoplaced yes)
-		(property "Reference" "#PWR02"
+		(property "Reference" "#PWR01"
 			(at 60.96 133.35 0)
 			(hide yes)
@@
 			(project "Power Supply ZensatV3"
 				(path "/6407b9bb-bcf3-46ce-88dc-7e023cbc9b7f"
-					(reference "#PWR02")
+					(reference "#PWR01")
 					(unit 1)
 				)
@@
 		(dnp no)
 		(fields_autoplaced yes)
-		(property "Reference" "U2"
+		(property "Reference" "U3"
 			(at 127.8733 128.27 0)
 			(show_name no)
@@
 			(project "Power Supply ZensatV3"
 				(path "/6407b9bb-bcf3-46ce-88dc-7e023cbc9b7f"
-					(reference "U2")
+					(reference "U3")
 					(unit 1)
 				)
@@
 		(dnp no)
 		(fields_autoplaced yes)
-		(property "Reference" "U3"
+		(property "Reference" "U1"
 			(at 65.6433 124.46 0)
 			(show_name no)
@@
 			(project "Power Supply ZensatV3"
 				(path "/6407b9bb-bcf3-46ce-88dc-7e023cbc9b7f"
-					(reference "U3")
+					(reference "U1")
 					(unit 1)
 				)
@@
 				)
 			)
-		)
-	)
-	(sheet
-		(at 179.07 62.23)
-		(size 25.4 19.05)
-		(exclude_from_sim no)
-		(in_bom yes)
-		(on_board yes)
-		(dnp no)
-		(fields_autoplaced yes)
-		(stroke
-			(width 0.1524)
-			(type solid)
-		)
-		(fill
-			(color 0 0 0 0)
-		)
-		(property "Sheetname" "5V Regulator"
-			(at 179.07 61.5184 0)
-			(show_name no)
-			(do_not_autoplace no)
-			(effects
-				(font
-					(size 1.27 1.27)
-				)
-				(justify left bottom)
-			)
-		)
-		(property "Sheetfile" "5vreg.kicad_sch"
-			(at 179.07 81.8646 0)
-			(show_name no)
-			(do_not_autoplace no)
-			(effects
-				(font
-					(size 1.27 1.27)
-				)
-				(justify left top)
-			)
-		)
-		(instances
-			(project "Power Supply ZensatV3"
-				(path "/6407b9bb-bcf3-46ce-88dc-7e023cbc9b7f"
-					(page "4")
-				)
-			)
-		)
-	)
-	(sheet
-		(at 179.07 33.02)
-		(size 25.4 19.05)
-		(exclude_from_sim no)
-		(in_bom yes)
-		(on_board yes)
-		(dnp no)
-		(fields_autoplaced yes)
-		(stroke
-			(width 0.1524)
-			(type solid)
-		)
-		(fill
-			(color 0 0 0 0)
-		)
-		(property "Sheetname" "3.3V Regulator"
-			(at 179.07 32.3084 0)
-			(show_name no)
-			(do_not_autoplace no)
-			(effects
-				(font
-					(size 1.27 1.27)
-				)
-				(justify left bottom)
-			)
-		)
-		(property "Sheetfile" "3V3Reg.kicad_sch"
-			(at 179.07 52.6546 0)
-			(show_name no)
-			(do_not_autoplace no)
-			(effects
-				(font
-					(size 1.27 1.27)
-				)
-				(justify left top)
-			)
-		)
-		(instances
-			(project "Power Supply ZensatV3"
-				(path "/6407b9bb-bcf3-46ce-88dc-7e023cbc9b7f"
-					(page "3")
-				)
-			)
