File: PCB Baterias/Kicad/PCB Bateria.kicad_sch (KiCad schematic)
At the start: 34 parts, among them J1 BatBus, J1 Conn_01x01_Socket, J2 Conn_01x02, J3 Conn_01x01_Socket, J4 Conn_01x01_Socket, J5 Conn_01x01_Socket, J6 Conn_01x01_Socket, J7 Conn_01x01_Socket, J8 Conn_01x01_Socket, J9 Conn_01x01_Socket, Q1 Si4162DY, Q2 Si4162DY, U7 INA3221

Commit message: borabill
Parts:
- added C1, C2: C_Small, symbol Device:C_Small
- added C33: 100nF 10V, Capacitor_SMD:C_0402_1005Metric_Pad0.74x0.62mm_HandSolder, symbol Device:C_Small
- added Q3, Q4: Si4162DY, Package_SO:SOIC-8_3.9x4.9mm_P1.27mm, symbol Transistor_FET:Si4162DY
- added R10, R8, R9: 10R, symbol Device:R
- added R31, R34, R38, R39: 10R, Resistor_SMD:R_0402_1005Metric_Pad0.72x0.64mm_HandSolder, symbol Device:R_Small
- added R40, R41, R42, R43: 0R, Resistor_SMD:R_0402_1005Metric_Pad0.72x0.64mm_HandSolder, symbol Device:R_Small
- added TH1: Thermistor_NTC, symbol Device:Thermistor_NTC
- added U1: LM75B, symbol Sensor_Temperature:LM75B
Connections:
- net +3.3V: now also C33.2, R40.2, R42.2, U1.8 (+Vs)
- net +BATT: now also R8.1
- net GND: now also C1.2, C33.1, Q4.5 (D), Q4.6 (D), Q4.7 (D), Q4.8 (D), R10.1, R41.2, R43.2, TH1.2, U1.4 (GND), U1.5 (A2); no longer J8.1 (Pin_1), J9.1 (Pin_1)
- net NTC: now also TH1.1
- net SCL: now also U1.2 (SCL)
- net SDA: now also U1.1 (SDA)
- net at Q2.5 (D), Q2.6 (D), Q2.7 (D)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: now also R39.2; no longer R5.2, R6.2, R7.2
- net at Q1.5 (D), Q1.6 (D), Q1.7 (D)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: now also R34.2; no longer J2.2 (Pin_2)
- net at J4.1 (Pin_1), J5.1 (Pin_1), J6.1 (Pin_1)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: now also R9.1
- new net: Q3.5 (D), Q3.6 (D), Q3.7 (D), Q3.8 (D), Q4.1 (S), Q4.2 (S), Q4.3 (S)
- new net: R40.1, R41.1, U1.7 (A0)
- new net: R38.2, R39.1
- new net: R42.1, R43.1, U1.6 (A1)
- new net: R38.1, R5.2, R6.2, R7.2
- new net: R31.2, R34.1
- new net: J2.2 (Pin_2), R31.1
- new net CS: R10.2
- new net OC: Q4.4 (G)
- new net OD: Q3.4 (G)
- new net VC: C2.1, R9.2
- new net VDD: C1.1, R8.2
- new net VSS: C2.2, J8.1 (Pin_1), J9.1 (Pin_1), Q3.1 (S), Q3.2 (S), Q3.3 (S)
- no-connect marks 4 -> 5
Other:
- note removed: "Resistores para escolha do endereço. Usar apenas 1."
- moved on the sheet: C31, C32, C34, C35, J1, J2, J3, J4, J5, J6, J7, J8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
