File: PCB Baterias/Kicad/PCB Bateria.kicad_sch (KiCad schematic)
At the start: 34 parts, among them J1 BatBus, J1 Conn_01x01_Socket, J2 Conn_01x02, J3 Conn_01x01_Socket, J4 Conn_01x01_Socket, J5 Conn_01x01_Socket, J6 Conn_01x01_Socket, J7 Conn_01x01_Socket, J8 Conn_01x01_Socket, J9 Conn_01x01_Socket, Q1 Si4162DY, Q2 Si4162DY, U7 INA3221

Commit message: Tomaz1
Parts:
- B1: renamed from J1; footprint (none) -> Connector_PinHeader_2.54mm:PinHeader_2x06_P2.54mm_Vertical_SMD
- J1, J3, J4, J5, J6, J7, J8, J9: footprint (none) -> Battery:BatteryClip_Keystone_54_D16-19mm
- J2: footprint (none) -> Connector_Molex:Molex_KK-254_AE-6410-02A_1x02_P2.54mm_Vertical
- R1, R2, R3, R4: footprint (none) -> Resistor_SMD:R_0805_2012Metric
- R5, R6, R7: footprint (none) -> Resistor_THT:R_Axial_DIN0516_L15.5mm_D5.0mm_P30.48mm_Horizontal
Other:
- moved on the sheet: J1
Changed lines of the file:
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@@
 	)
 	(junction
-		(at 57.15 134.62)
-		(diameter 0)
-		(color 0 0 0 0)
-	)
-	(junction
 		(at 114.3 91.44)
 		(diameter 0)
@@
 	)
 	(junction
+		(at 57.15 134.62)
+		(diameter 0)
+		(color 0 0 0 0)
+	)
+	(junction
 		(at 251.46 107.95)
 		(diameter 0)
@@
 	(wire
 		(pts
-			(xy 57.15 134.62) (xy 57.15 138.43)
+			(xy 63.5 134.62) (xy 63.5 139.7)
 		)
 		(stroke
@@
 	(wire
 		(pts
+			(xy 63.5 134.62) (xy 57.15 134.62)
+		)
+		(stroke
+			(width 0)
+			(type default)
+		)
+	)
+	(wire
+		(pts
 			(xy 173.99 120.65) (xy 173.99 124.46)
 		)
@@
 			)
 		)
-		(property "Footprint" ""
+		(property "Footprint" "Resistor_SMD:R_0805_2012Metric"
 			(at 243.84 109.728 90)
 			(hide yes)
@@
 			)
 		)
-		(property "Footprint" ""
+		(property "Footprint" "Resistor_THT:R_Axial_DIN0516_L15.5mm_D5.0mm_P30.48mm_Horizontal"
 			(at 264.922 88.9 90)
 			(hide yes)
@@
 			)
 		)
-		(property "Footprint" ""
+		(property "Footprint" "Battery:BatteryClip_Keystone_54_D16-19mm"
 			(at 58.42 167.64 0)
 			(hide yes)
@@
 			)
 		)
-		(property "Footprint" ""
+		(property "Footprint" "Resistor_SMD:R_0805_2012Metric"
 			(at 172.212 116.84 90)
 			(hide yes)
@@
 		(in_pos_files yes)
 		(dnp no)
-		(fields_autoplaced yes)
 		(property "Reference" "J3"
 			(at 45.72 141.6049 90)
@@
 		)
 		(property "Value" "Conn_01x01_Socket"
-			(at 45.72 144.1449 90)
+			(at 52.07 145.4149 90)
 			(show_name no)
 			(do_not_autoplace no)
@@
 			)
 		)
-		(property "Footprint" ""
+		(property "Footprint" "Battery:BatteryClip_Keystone_54_D16-19mm"
 			(at 44.45 143.51 0)
 			(hide yes)
@@
 			)
 		)
-		(property "Footprint" ""
+		(property "Footprint" "Battery:BatteryClip_Keystone_54_D16-19mm"
 			(at 58.42 154.94 0)
 			(hide yes)
@@
 			)
 		)
-		(property "Footprint" ""
+		(property "Footprint" "Battery:BatteryClip_Keystone_54_D16-19mm"
 			(at 44.45 154.94 0)
 			(hide yes)
@@
 			)
 		)
-		(property "Footprint" ""
+		(property "Footprint" "Connector_Molex:Molex_KK-254_AE-6410-02A_1x02_P2.54mm_Vertical"
 			(at 198.12 97.79 0)
 			(hide yes)
@@
 			)
 		)
-		(property "Footprint" ""
+		(property "Footprint" "Battery:BatteryClip_Keystone_54_D16-19mm"
 			(at 58.42 176.53 0)
 			(hide yes)
@@
 			)
 		)
-		(property "Footprint" ""
+		(property "Footprint" "Battery:BatteryClip_Keystone_54_D16-19mm"
 			(at 44.45 167.64 0)
 			(hide yes)
@@
 			)
 		)
-		(property "Footprint" ""
+		(property "Footprint" "Battery:BatteryClip_Keystone_54_D16-19mm"
 			(at 44.45 176.53 0)
 			(hide yes)
@@
 			)
 		)
-		(property "Footprint" ""
+		(property "Footprint" "Resistor_SMD:R_0805_2012Metric"
 			(at 166.37 112.268 90)
 			(hide yes)
@@
 	(symbol
 		(lib_id "Connector:Conn_01x01_Socket")
-		(at 57.15 143.51 270)
+		(at 63.5 144.78 270)
 		(unit 1)
 		(body_style 1)
@@
 		(in_pos_files yes)
 		(dnp no)
-		(fields_autoplaced yes)
 		(property "Reference" "J1"
-			(at 58.42 141.6049 90)
+			(at 66.04 142.24 90)
 			(show_name no)
 			(do_not_autoplace no)
@@
 		)
 		(property "Value" "Conn_01x01_Socket"
-			(at 58.42 144.1449 90)
+			(at 71.12 147.32 90)
+			(hide yes)
 			(show_name no)
 			(do_not_autoplace no)
@@
 			)
 		)
-		(property "Footprint" ""
-			(at 57.15 143.51 0)
+		(property "Footprint" "Battery:BatteryClip_Keystone_54_D16-19mm"
+			(at 63.5 144.78 0)
 			(hide yes)
 			(show_name no)
@@
 		)
 		(property "Datasheet" ""
-			(at 57.15 143.51 0)
+			(at 63.5 144.78 0)
 			(hide yes)
 			(show_name no)
@@
 		)
 		(property "Description" "Generic connector, single row, 01x01, script generated"
-			(at 57.15 143.51 0)
+			(at 63.5 144.78 0)
 			(hide yes)
 			(show_name no)
@@
 			)
 		)
-		(property "Footprint" ""
+		(property "Footprint" "Resistor_THT:R_Axial_DIN0516_L15.5mm_D5.0mm_P30.48mm_Horizontal"
 			(at 254.762 88.9 90)
 			(hide yes)
@@
 			)
 		)
-		(property "Footprint" ""
+		(property "Footprint" "Resistor_SMD:R_0805_2012Metric"
 			(at 249.682 114.3 90)
 			(hide yes)
@@
 		(dnp no)
 		(fields_autoplaced yes)
-		(property "Reference" "J1"
+		(property "Reference" "B1"
 			(at 260.35 16.51 0)
 			(show_name no)
@@
 			)
 		)
-		(property "Footprint" ""
+		(property "Footprint" "Connector_PinHeader_2.54mm:PinHeader_2x06_P2.54mm_Vertical_SMD"
 			(at 259.08 27.94 0)
 			(hide yes)
@@
 			(project "PCB Bateria"
 				(path "/971c4c7f-6281-4dec-89fa-5359e9e039dc"
-					(reference "J1")
+					(reference "B1")
 					(unit 1)
 				)
@@
 			)
 		)
-		(property "Footprint" ""
+		(property "Footprint" "Resistor_THT:R_Axial_DIN0516_L15.5mm_D5.0mm_P30.48mm_Horizontal"
 			(at 275.082 88.9 90)
 			(hide yes)
