File: PCB Baterias/Kicad/PCB Bateria.kicad_sch (KiCad schematic)
At the start: 34 parts, among them J1 BatBus, J1 Conn_01x01_Socket, J2 Conn_01x02, J3 Conn_01x01_Socket, J4 Conn_01x01_Socket, J5 Conn_01x01_Socket, J6 Conn_01x01_Socket, J7 Conn_01x01_Socket, J8 Conn_01x01_Socket, J9 Conn_01x01_Socket, Q1 Si4162DY, Q2 Si4162DY, U7 INA3221

Commit message: Main Board V1.0
Conclusão da Main Board.
Parts:
- renumbered J1 to B1
Changed lines of the file:
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@@
 	)
 	(junction
-		(at 57.15 134.62)
-		(diameter 0)
-		(color 0 0 0 0)
-	)
-	(junction
 		(at 114.3 91.44)
 		(diameter 0)
@@
 	)
 	(junction
+		(at 57.15 134.62)
+		(diameter 0)
+		(color 0 0 0 0)
+	)
+	(junction
 		(at 45.72 93.98)
 		(diameter 0)
@@
 		(dnp no)
 		(fields_autoplaced yes)
-		(property "Reference" "J1"
+		(property "Reference" "B1"
 			(at 260.35 16.51 0)
 			(show_name no)
@@
 			(project "PCB Bateria"
 				(path "/971c4c7f-6281-4dec-89fa-5359e9e039dc"
-					(reference "J1")
+					(reference "B1")
 					(unit 1)
 				)
