File: PCB Baterias/Kicad/PCB Bateria 09082026.kicad_pcb (KiCad board)
At the start: 2 copper layers, 86 x 86 mm, 52 parts, among them J1 Conn_Deploy, J2 18650 Socket, J3 18650 Socket, J4 18650 Socket, J5 18650 Socket, J6 18650 Socket, J7 18650 Socket, J8 18650 Socket, J9 18650 Socket, Q1 Si4162DY, Q2 Si4162DY, Q3 Si4162DY, Q4 Si4162DY, U1 INA3221, U2 MCP9808, U3 FM7021DB

Commit message: Final V1.0
Finalização da primeira versão.
Parts:
- removed R10, R14: 0R, Resistor_SMD:R_0402_1005Metric_Pad0.72x0.64mm_HandSolder
- added C8: 10uF 10V, Capacitor_SMD:C_0805_2012Metric_Pad1.18x1.45mm_HandSolder, B.Cu at (149.9, 109.8)
- added G***: LOGO, LOGO, F.Cu at (149.0, 102.8)
- added G***: LOGO, LogosZenith:Logo_29,1mm, F.Cu at (149.1, 63.0)
- added G***: LOGO, LogosZenith:Logo_29,1mm, B.Cu at (149.1, 63.0)
- added G***: LOGO, LOGO, B.Cu at (149.0, 82.9)
- added G***: LOGO, LOGO, B.Cu at (156.4, 114.6)
- added J2: PwrON, Connector_PinHeader_2.54mm:PinHeader_1x02_P2.54mm_Vertical, F.Cu at (111.5, 74.0)
- C6, C7, Q3, Q4, R21, R26, U3: moved to B.Cu
- R18: renamed from R20; moved to B.Cu
- R19: renamed from R18; moved to B.Cu
- R20: renamed from R19; moved to B.Cu
- R27: footprint Resistor_SMD:R_01005_0402Metric_Pad0.57x0.30mm_HandSolder -> Resistor_SMD:R_0402_1005Metric_Pad0.72x0.64mm_HandSolder; moved to B.Cu
- TH1: footprint Varistor:RV_Disc_D7mm_W3.4mm_P5mm -> Resistor_THT:R_Axial_DIN0204_L3.6mm_D1.6mm_P1.90mm_Vertical
- moved R18 49.6 mm to (130.1, 109.6), turned to 180 degrees
- moved R19 46.8 mm to (130.0, 117.6), turned to -90 degrees
- moved TH1 44.3 mm to (168.3, 94.1), turned to 90 degrees
- moved R27 42.2 mm to (150.4, 105.1), turned to 90 degrees
- moved R20 41.8 mm to (168.0, 117.6), turned to -90 degrees
- moved C6 34.1 mm to (161.5, 92.7), turned to 180 degrees
- moved C7 33.8 mm to (160.3, 94.9), turned to 180 degrees
- moved R26 33.6 mm to (130.5, 97.0), turned to 90 degrees
- moved Q3 32.5 mm to (164.0, 106.4), turned to 180 degrees
- moved Q2 32.0 mm to (165.6, 123.8)
- moved Q1 31.7 mm to (132.4, 123.8)
- moved R24 31.3 mm to (137.0, 125.1), turned to 90 degrees
- moved R25 31.3 mm to (161.0, 122.6), turned to -90 degrees
- moved R23 28.9 mm to (159.6, 122.6), turned to 90 degrees
- moved R22 28.2 mm to (138.4, 125.1), turned to -90 degrees
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- renumbered J9 to J10, J2 to J3, J3 to J4, J4 to J5, J5 to J6, J6 to J7, J7 to J8, J8 to J9
Connections:
- J3 pad 1: /BATT_Sense -> Net-(J2-Pin_2)
- J4 pad 1: /BATT_Sense -> Net-(J2-Pin_2)
- R21 pad 1: /BATT_Sense -> Net-(J2-Pin_2)
Routing:
- net Net-(J10-Pin_1): track 13.8 -> 98.6 mm
- net /Heater_Sense+: track 30.7 -> 112.4 mm, vias 1 -> 2
- net /Deploy_Sense+: track 1.29 -> 76.3 mm, vias 0 -> 2
- net /BATT_Sense: track 0.00 -> 74.0 mm, vias 0 -> 2
- net Net-(J2-Pin_2): track 0.00 -> 69.9 mm
- net /Heater_Sense-: track 0.00 -> 69.5 mm, vias 0 -> 2
- net +3.3VP: track 25.2 -> 88.6 mm, vias 2 -> 3
- net /I2C2_SCL: track 4.56 -> 61.1 mm, vias 0 -> 3
- net Net-(Q1-G): track 55.9 -> 3.54 mm
- net Net-(J5-Pin_1): track 225.3 -> 180.5 mm, vias 2 -> 0
- net /NTC: track 0.00 -> 44.6 mm, vias 0 -> 1
- net /I2C2_SDA: track 11.5 -> 55.7 mm, vias 0 -> 1
- net Net-(U3-VDD): track 0.00 -> 42.2 mm
- net Net-(U3-VC): track 0.00 -> 40.1 mm
- net (no net): track 34.5 -> 0.00 mm
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- added copper zone on B.Cu, net /Deploy_Sense-
- added copper zone on B.Cu, net /Heater_Sense-
- added copper zone on B.Cu, net GND
- added copper zone on B.Cu, net Net-(Q3-D-Pad5)
- added copper zone on F.Cu, net Net-(Q3-D-Pad5)
Other:
- copper layers 2 -> 4
- board text added: "22/10/2026"
