File: PCB Baterias/Kicad/PCB Bateria 09082026.kicad_sch (KiCad schematic)
At the start: 53 parts, among them J1 Conn_Deploy, J10 PwrON, J2 18650 Socket, J3 18650 Socket, J4 18650 Socket, J5 18650 Socket, J6 18650 Socket, J7 18650 Socket, J8 18650 Socket, J9 18650 Socket, Q1 Si4162DY, Q2 Si4162DY, Q3 Si4162DY, Q4 Si4162DY, U1 INA3221, U2 MCP9808, U3 FM7021DB

Commit message: Final V1.0
Finalização da primeira versão.
Parts:
- removed R10, R14: 0R, Resistor_SMD:R_0402_1005Metric_Pad0.72x0.64mm_HandSolder, symbol Device:R_Small
- added C8: 10uF 10V, Capacitor_SMD:C_0805_2012Metric_Pad1.18x1.45mm_HandSolder, symbol Device:C_Small
- J2: renamed from J10; footprint (none) -> Connector_PinHeader_2.54mm:PinHeader_1x02_P2.54mm_Vertical
- R27: footprint Resistor_SMD:R_01005_0402Metric_Pad0.57x0.30mm_HandSolder -> Resistor_SMD:R_0402_1005Metric_Pad0.72x0.64mm_HandSolder
- TH1: footprint Varistor:RV_Disc_D7mm_W3.4mm_P5mm -> Resistor_THT:R_Axial_DIN0204_L3.6mm_D1.6mm_P1.90mm_Vertical
- renumbered J9 to J10, J2 to J3, J3 to J4, J4 to J5, J5 to J6, J6 to J7, J7 to J8, J8 to J9, R20 to R18, R18 to R19, R19 to R20
Connections:
- net +3.3VP: now also C8.1
- net +BATT: now also R18.1; no longer J2.1 (Pin_1)
- net BATT_Sense: now also J2.1 (Pin_1); no longer J3.1 (Pin_1), J4.1 (Pin_1), R21.1
- net GND: now also C8.2
- net at J2.2 (Pin_2): now also J3.1 (Pin_1), J4.1 (Pin_1), R21.1; no longer R18.1
Other:
- moved on the sheet: J2, R18
