File: Main Board/Kicad/Power Supply ZensatV3.kicad_pcb (KiCad board)
At the start: 2 copper layers, 86 x 86 mm, 24 parts, among them J1 ZenBus, U1 STM32L476RGTx, U2 INA3221, U3 INA3221, U4 LMR33630ADDA, U5 LT3652IMSE, U6 LMR33630ADDA, U7 AMS1117-3.3

Commit message: Atualização do circuito/pcb
Parts:
- added C11: 22uF, Capacitor_SMD:C_1206_3216Metric_Pad1.33x1.80mm_HandSolder, F.Cu at (118.5, 72.8)
- added C12: 22uF, Capacitor_SMD:C_1206_3216Metric_Pad1.33x1.80mm_HandSolder, F.Cu at (118.5, 75.3)
- added C13: 22uF, Capacitor_SMD:C_1206_3216Metric_Pad1.33x1.80mm_HandSolder, F.Cu at (118.5, 77.8)
- added C14: 1uF, Capacitor_SMD:C_0402_1005Metric_Pad0.74x0.62mm_HandSolder, F.Cu at (130.1, 82.5)
- added C15: 100nF, Capacitor_SMD:C_0402_1005Metric_Pad0.74x0.62mm_HandSolder, F.Cu at (173.8, 101.2)
- added C16: 10uF, Capacitor_SMD:C_1206_3216Metric_Pad1.33x1.80mm_HandSolder, F.Cu at (180.2, 100.2)
- added C17: 10uF, Capacitor_SMD:C_1206_3216Metric_Pad1.33x1.80mm_HandSolder, F.Cu at (179.6, 69.4)
- added C18: 1uF, Capacitor_SMD:C_0402_1005Metric_Pad0.74x0.62mm_HandSolder, F.Cu at (179.9, 76.5)
- added C19: 10uF, Capacitor_SMD:C_1206_3216Metric_Pad1.33x1.80mm_HandSolder, F.Cu at (179.6, 72.8)
- added C20: 680nF, Capacitor_SMD:C_0402_1005Metric_Pad0.74x0.62mm_HandSolder, F.Cu at (179.9, 78.5)
- added D1: 1N5819HW, Diode_SMD:D_SOD-123, F.Cu at (162.8, 69.4)
- added D2: 1N5819HW, Diode_SMD:D_SOD-123, F.Cu at (162.8, 72.8)
- added D3: 1N5819HW, Diode_SMD:D_SOD-123, F.Cu at (162.8, 76.1)
- added D4: MBRS340, Diode_SMD:D_SMC, F.Cu at (154.9, 106.0)
- added D5: 1N5819HW, Diode_SMD:D_SOD-123, F.Cu at (162.8, 79.5)
- added D6: 1N5819HW, Diode_SMD:D_SOD-123, F.Cu at (142.1, 104.3)
- added L3: 47uH, Inductor_SMD:L_TDK_SLF7032, F.Cu at (147.2, 109.3)
- added R1: R05, Resistor_SMD:R_0612_1632Metric_Pad1.18x3.40mm_HandSolder, F.Cu at (141.7, 67.1)
- added R10: R_Small, Resistor_SMD:R_0402_1005Metric_Pad0.72x0.64mm_HandSolder, F.Cu at (176.7, 80.5)
- added R11: 626k, Resistor_SMD:R_0402_1005Metric_Pad0.72x0.64mm_HandSolder, F.Cu at (176.7, 82.5)
- added R12: 412k, Resistor_SMD:R_0402_1005Metric_Pad0.72x0.64mm_HandSolder, F.Cu at (153.4, 97.8)
- added R6: 14,9k, Resistor_SMD:R_0402_1005Metric_Pad0.72x0.64mm_HandSolder, F.Cu at (129.4, 84.7)
- added R7: R_Small, Resistor_SMD:R_0402_1005Metric_Pad0.72x0.64mm_HandSolder, F.Cu at (176.7, 76.5)
- added R8: 0R33, Resistor_SMD:R_1210_3225Metric_Pad1.30x2.65mm_HandSolder, F.Cu at (141.1, 108.2)
- added R9: 1k, Resistor_SMD:R_0402_1005Metric_Pad0.72x0.64mm_HandSolder, F.Cu at (176.7, 78.5)
- added U8: LM234DT, Package_SO:SOIC-8_3.9x4.9mm_P1.27mm, F.Cu at (167.9, 92.7)
- added U9: LT3652IMSE, Package_SO:MSOP-12-1EP_3x4.039mm_P0.65mm_EP1.651x2.845mm_ThermalVias, F.Cu at (147.1, 102.3)
- C2, C9: value 22uF -> 10uF
- C6: value 100nF -> 22uF; footprint Capacitor_SMD:C_0402_1005Metric_Pad0.74x0.62mm_HandSolder -> Capacitor_SMD:C_1206_3216Metric_Pad1.33x1.80mm_HandSolder
- C7: value 22uF -> 1uF; footprint Capacitor_SMD:C_1206_3216Metric_Pad1.33x1.80mm_HandSolder -> Capacitor_SMD:C_0402_1005Metric_Pad0.74x0.62mm_HandSolder
- C8: value 22uF -> 100nF; footprint Capacitor_SMD:C_1206_3216Metric_Pad1.33x1.80mm_HandSolder -> Capacitor_SMD:C_0402_1005Metric_Pad0.74x0.62mm_HandSolder
- R2, R5: value R_Small -> 100k
- R3: value R_Small -> 43,2k
- R4: value R_Small -> R05; footprint Resistor_SMD:R_0402_1005Metric_Pad0.72x0.64mm_HandSolder -> Resistor_SMD:R_0612_1632Metric_Pad1.18x3.40mm_HandSolder
- U2, U3: value INA3221 -> LMR33630ADDA; footprint Package_DFN_QFN:Texas_RGV0016A_VQFN-16-1EP_4x4mm_P0.65mm_EP2.1x2.1mm -> Package_SO:Texas_HSOP-8-1EP_3.9x4.9mm_P1.27mm_ThermalVias
- U4: value LMR33630ADDA -> AMS1117-3.3; footprint Package_SO:Texas_HSOP-8-1EP_3.9x4.9mm_P1.27mm_ThermalVias -> Package_TO_SOT_SMD:SOT-223-3_TabPin2
- U5: value LT3652IMSE -> INA3221; footprint Package_SO:MSOP-12-1EP_3x4.039mm_P0.65mm_EP1.651x2.845mm_ThermalVias -> Package_DFN_QFN:Texas_RGV0016A_VQFN-16-1EP_4x4mm_P0.65mm_EP2.1x2.1mm
- U6: value LMR33630ADDA -> INA3221; footprint Package_SO:Texas_HSOP-8-1EP_3.9x4.9mm_P1.27mm_ThermalVias -> Package_DFN_QFN:Texas_RGV0016A_VQFN-16-1EP_4x4mm_P0.65mm_EP2.1x2.1mm
- U7: value AMS1117-3.3 -> INA3221; footprint Package_TO_SOT_SMD:SOT-223-3_TabPin2 -> Package_DFN_QFN:Texas_RGV0016A_VQFN-16-1EP_4x4mm_P0.65mm_EP2.1x2.1mm
- moved U4 57.8 mm to (175.5, 109.0), turned to -90 degrees
- moved U3 40.0 mm to (125.0, 81.8)
- moved R4 34.2 mm to (121.0, 67.2)
- moved U5 27.7 mm to (115.9, 94.6), turned to -90 degrees
- moved U7 27.6 mm to (127.4, 94.5), turned to -90 degrees
- moved R3 26.0 mm to (150.3, 84.5), turned to 90 degrees
- moved C5 26.0 mm to (139.2, 72.7)
- moved C4 24.3 mm to (139.2, 75.2)
- moved C1 24.0 mm to (150.3, 80.3)
- moved L1 23.9 mm to (146.2, 75.2)
- moved C3 23.7 mm to (139.2, 77.7)
- moved C2 23.1 mm to (137.9, 81.7), turned to -90 degrees
- moved R2 22.1 mm to (148.5, 85.1), turned to 0 degrees
- moved C10 21.6 mm to (118.5, 70.3)
- moved U2 19.0 mm to (145.9, 81.6)
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Connections:
- net /Main PCB/3V3 renamed +3V3
- net /Main PCB/CAN_H renamed BUS_CAN_H
- net /Main PCB/CAN_L renamed BUS_CAN_L
- net /Main PCB/MISO renamed BUS_MISO
- net /Main PCB/MOSI renamed BUS_MOSI
- net /Main PCB/SCL renamed BUS_SCL
- net /Main PCB/SCLK renamed BUS_SCLK
- net /Main PCB/SDA renamed BUS_SDA
- net /Main PCB/SOL+ renamed SOL+
- net /Main PCB/SOL- renamed SOL-
- C1 pad 1: Net-(U4-BOOT) -> Net-(U2-BOOT)
- C1 pad 2: Net-(U4-SW) -> Net-(U2-SW)
- C10 pad 2: /Regulators/5V -> /Regulators/+5V_Sense
- C2 pad 2: /Regulators/3V3 -> BAT+
- C3 pad 2: /Regulators/3V3 -> /Regulators/+3V3_Sense
- C4 pad 2: /Regulators/3V3 -> /Regulators/+3V3_Sense
- C5 pad 2: /Regulators/3V3 -> /Regulators/+3V3_Sense
- C6 pad 1: Net-(U6-BOOT) -> GND
- C6 pad 2: Net-(U6-SW) -> /Regulators/+3V3_Sense
- C7 pad 2: /Regulators/5V -> Net-(U2-VCC)
- C8 pad 1: GND -> Net-(U3-BOOT)
- C8 pad 2: /Regulators/5V -> Net-(U3-SW)
- C9 pad 2: /Regulators/5V -> BAT+
- J1 pad 10: /Main PCB/5V -> +5V
- J1 pad 5: /Main PCB/BAT+ -> BAT+
- J1 pad 6: /Main PCB/BAT+ -> BAT+
- J1 pad 9: /Main PCB/5V -> +5V
- L1 pad 1: Net-(U4-SW) -> Net-(U2-SW)
- L1 pad 2: /Regulators/3V3 -> /Regulators/+3V3_Sense
- L2 pad 1: Net-(U6-SW) -> Net-(U3-SW)
- L2 pad 2: /Regulators/5V -> /Regulators/+5V_Sense
- R2 pad 1: /Regulators/3V3 -> /Regulators/+3V3_Sense
- R2 pad 2: Net-(U4-FB) -> Net-(U2-FB)
- R3 pad 1: Net-(U4-FB) -> Net-(U2-FB)
- R4 pad 1: /Regulators/5V -> /Regulators/+5V_Sense
- R4 pad 2: Net-(U6-FB) -> +5V
- R5 pad 1: Net-(U6-FB) -> /Regulators/+5V_Sense
- R5 pad 2: GND -> Net-(U3-FB)
- U2 pad 1: unconnected-(U2-IN-3-Pad1) -> GND
- U2 pad 2: unconnected-(U2-IN+3-Pad2) -> BAT+
- U2 pad 3: GND -> /Regulators/+3V3_Enable
- U2 pad 4: unconnected-(U2-VS-Pad4) -> /Regulators/+3V3_PG
- U2 pad 5: unconnected-(U2-A0-Pad5) -> Net-(U2-FB)
- U2 pad 6: unconnected-(U2-SCL-Pad6) -> Net-(U2-VCC)
- U2 pad 7: unconnected-(U2-SDA-Pad7) -> Net-(U2-BOOT)
- U2 pad 8: unconnected-(U2-WARNING-Pad8) -> Net-(U2-SW)
- U2 pad 9: unconnected-(U2-CRITICAL-Pad9) -> GND
- U3 pad 1: unconnected-(U3-IN-3-Pad1) -> GND
- U3 pad 2: unconnected-(U3-IN+3-Pad2) -> BAT+
- U3 pad 3: GND -> /Regulators/+5V_Enable
- U3 pad 4: unconnected-(U3-VS-Pad4) -> /Regulators/+5V_PG
- U3 pad 5: unconnected-(U3-A0-Pad5) -> Net-(U3-FB)
- U3 pad 6: unconnected-(U3-SCL-Pad6) -> Net-(U3-VCC)
- U3 pad 7: unconnected-(U3-SDA-Pad7) -> Net-(U3-BOOT)
- U3 pad 8: unconnected-(U3-WARNING-Pad8) -> Net-(U3-SW)
- U3 pad 9: unconnected-(U3-CRITICAL-Pad9) -> GND
- U4 pad 2: /Regulators/BAT+ -> +3.3VP
- U4 pad 3: /Regulators/BAT+ -> BATC+
- U5 pad 3: unconnected-(U5-~{SHDN}-Pad3) -> GND
- U6 pad 1: GND -> unconnected-(U6-IN-3-Pad1)
- U6 pad 2: /Regulators/BAT+ -> unconnected-(U6-IN+3-Pad2)
- U6 pad 3: /Regulators/BAT+ -> GND
- U6 pad 5: Net-(U6-FB) -> unconnected-(U6-A0-Pad5)
- U6 pad 7: Net-(U6-BOOT) -> unconnected-(U6-SDA-Pad7)
- U6 pad 8: Net-(U6-SW) -> unconnected-(U6-WARNING-Pad8)
- U6 pad 9: GND -> unconnected-(U6-CRITICAL-Pad9)
- U7 pad 1: GND -> unconnected-(U7-IN-3-Pad1)
- U7 pad 3: /Regulators/BAT+ -> GND
Routing:
- net +5V: track 0.00 -> 16.1 mm
- net /Regulators/+3V3_Sense: track 0.00 -> 13.7 mm, vias 0 -> 2
- net +3V3: track 0.00 -> 12.8 mm
- net Net-(U2-FB): track 0.00 -> 3.14 mm
- net Net-(U3-FB): track 0.00 -> 3.00 mm
- net Net-(U2-BOOT): track 0.00 -> 1.95 mm
- net Net-(U2-VCC): track 0.00 -> 1.81 mm
- net Net-(U3-VCC): track 0.00 -> 1.76 mm
- net Net-(U3-BOOT): track 0.00 -> 1.76 mm
- added copper zone on F.Cu, net /Regulators/+3V3_Sense
- added copper zone on F.Cu, net /Regulators/+5V_Sense
- added copper zone on F.Cu, net GND
- added copper zone on F.Cu, net Net-(U2-SW)
- added copper zone on F.Cu, net Net-(U3-SW)
Other:
- copper layers 2 -> 4

Commit message: atualização pcb
Parts:
- removed the U5 at (115.9, 94.6)
- removed the U7 at (127.4, 94.5)
- added C1: 100nF, Capacitor_SMD:C_0402_1005Metric_Pad0.74x0.62mm_HandSolder, F.Cu at (137.1, 100.8)
- added C2: 100nF, Capacitor_SMD:C_0402_1005Metric_Pad0.74x0.62mm_HandSolder, F.Cu at (141.3, 89.2)
- added C21: 100nF, Capacitor_SMD:C_0402_1005Metric_Pad0.74x0.62mm_HandSolder, F.Cu at (149.3, 69.0)
- added C3: 100nF, Capacitor_SMD:C_0402_1005Metric_Pad0.74x0.62mm_HandSolder, F.Cu at (154.1, 94.8)
- added C4: 100nF, Capacitor_SMD:C_0402_1005Metric_Pad0.74x0.62mm_HandSolder, F.Cu at (149.8, 89.2)
- added J2: Conn_01x02_Pin, Connector_JST:JST_ZH_B2B-ZR_1x02_P1.50mm_Vertical, F.Cu at (108.7, 72.5)
- added J3: Conn_01x02_Pin, Connector_JST:JST_ZH_B2B-ZR_1x02_P1.50mm_Vertical, F.Cu at (182.5, 74.2)
- added J4: Conn_01x02_Pin, Connector_JST:JST_ZH_B2B-ZR_1x02_P1.50mm_Vertical, F.Cu at (108.8, 120.8)
- added J5: Conn_01x02_Pin, Connector_JST:JST_ZH_B2B-ZR_1x02_P1.50mm_Vertical, F.Cu at (182.3, 122.2)
- added JP1: SolderJumper_2_Open, Jumper:SolderJumper-2_P1.3mm_Open_RoundedPad1.0x1.5mm, F.Cu at (129.4, 100.2)
- added JP2: SolderJumper_2_Open, Jumper:SolderJumper-2_P1.3mm_Open_RoundedPad1.0x1.5mm, F.Cu at (125.8, 100.2)
- added JP3: SolderJumper_2_Open, Jumper:SolderJumper-2_P1.3mm_Open_RoundedPad1.0x1.5mm, F.Cu at (122.3, 100.2)
- added JP4: SolderJumper_2_Open, Jumper:SolderJumper-2_P1.3mm_Open_RoundedPad1.0x1.5mm, F.Cu at (118.6, 100.2)
- added JP5: SolderJumper_2_Open, Jumper:SolderJumper-2_P1.3mm_Open_RoundedPad1.0x1.5mm, F.Cu at (115.3, 100.2)
- added R10: 10k, Resistor_SMD:R_0402_1005Metric_Pad0.72x0.64mm_HandSolder, F.Cu at (141.1, 71.8)
- added R11: 0R33, Resistor_SMD:R_1210_3225Metric_Pad1.30x2.65mm_HandSolder, F.Cu at (135.8, 114.8)
- added R7: 10k, Resistor_SMD:R_0402_1005Metric_Pad0.72x0.64mm_HandSolder, F.Cu at (141.1, 69.5)
- added R8: 10k, Resistor_SMD:R_0402_1005Metric_Pad0.72x0.64mm_HandSolder, F.Cu at (141.1, 68.2)
- added R9: 10k, Resistor_SMD:R_0402_1005Metric_Pad0.72x0.64mm_HandSolder, F.Cu at (141.1, 67.0)
- added U2: SN65HVD230, Package_SO:SOIC-8_3.9x4.9mm_P1.27mm, F.Cu at (145.6, 81.8)
- C11: renamed from C7; footprint Capacitor_SMD:C_0402_1005Metric_Pad0.74x0.62mm_HandSolder -> Capacitor_SMD:C_0603_1608Metric_Pad1.08x0.95mm_HandSolder
- C13: renamed from C9; footprint Capacitor_SMD:C_1206_3216Metric_Pad1.33x1.80mm_HandSolder -> Capacitor_SMD:C_0805_2012Metric_Pad1.18x1.45mm_HandSolder
- C18: renamed from C14; footprint Capacitor_SMD:C_0402_1005Metric_Pad0.74x0.62mm_HandSolder -> Capacitor_SMD:C_0603_1608Metric_Pad1.08x0.95mm_HandSolder
- C20: renamed from C16; footprint Capacitor_SMD:C_1206_3216Metric_Pad1.33x1.80mm_HandSolder -> Capacitor_SMD:C_0805_2012Metric_Pad1.18x1.45mm_HandSolder
- C22: renamed from C17; footprint Capacitor_SMD:C_1206_3216Metric_Pad1.33x1.80mm_HandSolder -> Capacitor_SMD:C_0805_2012Metric_Pad1.18x1.45mm_HandSolder
- C23: renamed from C18; value 1uF -> 1uF 50V; footprint Capacitor_SMD:C_0402_1005Metric_Pad0.74x0.62mm_HandSolder -> Capacitor_SMD:C_0603_1608Metric_Pad1.08x0.95mm_HandSolder
- C6: renamed from C2; footprint Capacitor_SMD:C_1206_3216Metric_Pad1.33x1.80mm_HandSolder -> Capacitor_SMD:C_0805_2012Metric_Pad1.18x1.45mm_HandSolder
- D4: value MBRS340 -> SS34; footprint Diode_SMD:D_SMC -> Diode_SMD:D_SMA
- moved D3 68.1 mm to (108.5, 117.2), turned to 180 degrees
- moved C22 63.2 mm to (138.6, 117.5)
- moved C25 61.4 mm to (139.1, 124.2)
- moved R12 58.7 mm to (137.1, 119.8), turned to 90 degrees
- moved R14 58.1 mm to (135.8, 119.8), turned to 90 degrees
- moved R15 57.5 mm to (137.1, 122.1), turned to 90 degrees
- moved C23 55.4 mm to (145.3, 119.8), turned to -90 degrees
- moved D1 55.1 mm to (108.2, 77.5), turned to 180 degrees
- moved C24 53.5 mm to (159.3, 122.2)
- moved R16 53.0 mm to (144.1, 124.2)
- moved U7 45.5 mm to (132.3, 121.0), turned to -90 degrees
- moved D6 42.7 mm to (182.8, 117.2)
- moved R17 28.9 mm to (141.8, 124.2), turned to 0 degrees
- moved U6 26.9 mm to (145.5, 70.0), turned to 180 degrees
- moved C20 26.1 mm to (155.6, 108.8)
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- renumbered C6 to C10, C8 to C12, C10 to C14, C11 to C15, C12 to C16, C13 to C17, C15 to C19, C19 to C24, C20 to C25, C1 to C5, C3 to C7, C4 to C8, C5 to C9, D6 to D5, D5 to D6, R7 to R12, R8 to R13, R9 to R14, R10 to R15, R11 to R16, R12 to R17, U2 to U3, U3 to U4, U4 to U5, U8 to U7, U9 to U8
Connections:
- C10 pad 2: /Regulators/+3V3_Sense -> +3V3_Sense
- C14 pad 2: /Regulators/+5V_Sense -> +5V_Sense
- C15 pad 2: /Regulators/+5V_Sense -> +5V_Sense
- C16 pad 2: /Regulators/+5V_Sense -> +5V_Sense
- C17 pad 2: /Regulators/+5V_Sense -> +5V_Sense
- C19 pad 2: BATC+ -> BAT+
- C22 pad 1: Net-(D1-K) -> -SOL_Sense
- C7 pad 2: /Regulators/+3V3_Sense -> +3V3_Sense
- C8 pad 2: /Regulators/+3V3_Sense -> +3V3_Sense
- C9 pad 2: /Regulators/+3V3_Sense -> +3V3_Sense
- D1 pad 1: Net-(D1-K) -> +SOL_Sense
- D1 pad 2: /Charger/SOL1 -> Net-(D1-A)
- D2 pad 1: Net-(D1-K) -> +SOL_Sense
- D2 pad 2: /Charger/SOL2 -> Net-(D2-A)
- D3 pad 1: Net-(D1-K) -> +SOL_Sense
- D3 pad 2: /Charger/SOL3 -> Net-(D3-A)
- D6 pad 1: Net-(D1-K) -> +SOL_Sense
- D6 pad 2: /Charger/SOL4 -> Net-(D6-A)
- L1 pad 2: /Regulators/+3V3_Sense -> +3V3_Sense
- L2 pad 2: /Regulators/+5V_Sense -> +5V_Sense
- R1 pad 1: /Regulators/+3V3_Sense -> +3V3_Sense
- R12 pad 2: Net-(D1-K) -> -SOL_Sense
- R2 pad 1: /Regulators/+3V3_Sense -> +3V3_Sense
- R4 pad 1: /Regulators/+5V_Sense -> +5V_Sense
- R5 pad 1: /Regulators/+5V_Sense -> +5V_Sense
- U1 pad 13: unconnected-(U1-VDDA-Pad13) -> +3.3VP
- U1 pad 19: unconnected-(U1-VDD-Pad19) -> +3.3VP
- U1 pad 32: unconnected-(U1-VDD-Pad32) -> +3.3VP
- U1 pad 48: unconnected-(U1-VDDUSB-Pad48) -> +3.3VP
- U1 pad 64: unconnected-(U1-VDD-Pad64) -> +3.3VP
- U5 pad 3: BATC+ -> BAT+
- U6 pad 1: unconnected-(U6-IN-3-Pad1) -> +3V3
- U6 pad 10: unconnected-(U6-PV-Pad10) -> /Monitor/PV
- U6 pad 11: unconnected-(U6-IN-1-Pad11) -> +5V
- U6 pad 12: unconnected-(U6-IN+1-Pad12) -> +5V_Sense
- U6 pad 13: unconnected-(U6-TC-Pad13) -> /Monitor/TC
- U6 pad 14: unconnected-(U6-IN-2-Pad14) -> -SOL_Sense
- U6 pad 15: unconnected-(U6-IN+2-Pad15) -> +SOL_Sense
- U6 pad 16: unconnected-(U6-VPU-Pad16) -> Net-(JP1-A)
- U6 pad 17: unconnected-(U6-EP-Pad17) -> GND
- U6 pad 2: unconnected-(U6-IN+3-Pad2) -> +3V3_Sense
- U6 pad 4: unconnected-(U6-VS-Pad4) -> +3.3VP
- U6 pad 5: unconnected-(U6-A0-Pad5) -> Net-(JP2-A)
- U6 pad 6: unconnected-(U6-SCL-Pad6) -> /Monitor/SCL
- U6 pad 7: unconnected-(U6-SDA-Pad7) -> /Monitor/SDA
- U6 pad 8: unconnected-(U6-WARNING-Pad8) -> /Monitor/WARNING
- U6 pad 9: unconnected-(U6-CRITICAL-Pad9) -> /Monitor/CRITICAL
- U7 pad 4: Net-(D1-K) -> -SOL_Sense
- U8 pad 1: Net-(D1-K) -> -SOL_Sense
- U8 pad 3: Net-(D1-K) -> unconnected-(U8-~{SHDN}-Pad3)
Routing:
- net +5V_Sense: track 0.00 -> 29.7 mm, vias 0 -> 2
- net +3V3_Sense: track 0.00 -> 27.4 mm, vias 0 -> 2
- net +3.3VP: track 0.00 -> 23.6 mm, vias 0 -> 4
- net /Regulators/+3V3_Sense: track 13.7 -> 0.00 mm, vias 2 -> 0
- net Net-(U8-V_{IN_REG}): track 0.00 -> 10.3 mm
- net -SOL_Sense: track 0.00 -> 9.21 mm
- net /Monitor/WARNING: track 0.00 -> 3.35 mm
- net /Monitor/TC: track 0.00 -> 2.92 mm
- net Net-(JP1-A): track 0.00 -> 2.53 mm, vias 0 -> 2
- net +3V3: track 12.8 -> 15.2 mm, vias 0 -> 3
- net /Monitor/CRITICAL: track 0.00 -> 2.31 mm
- net Net-(D5-K): track 0.00 -> 2.24 mm
- net Net-(U8-V_{FB}): track 0.00 -> 2.18 mm
- net /Monitor/PV: track 0.00 -> 2.06 mm
- net GND: track 0.00 -> 2.00 mm, vias 0 -> 111
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- added copper zone on F.Cu, net +3V3_Sense
- added copper zone on F.Cu, net +5V_Sense
- added copper zone on F.Cu, net -SOL_Sense
- added copper zone on F.Cu, net BAT+
- added copper zone on B.Cu, net GND
- added copper zone on In1.Cu, net GND
- added copper zone on F.Cu, net Net-(D4-K)
- added copper zone on F.Cu, net Net-(D5-K)
- added copper zone on F.Cu, net Net-(U8-SENSE)
- removed copper zone on F.Cu, net /Regulators/+3V3_Sense
- removed copper zone on F.Cu, net /Regulators/+5V_Sense
Other:
- board text added: "+3.3V"
- board text added: "+5V"
- board text added: "Solar MPPT & Charger"

Commit message: atualização pcb
Parts:
- removed JP3, JP4, JP5: SolderJumper_2_Open, Jumper:SolderJumper-2_P1.3mm_Open_RoundedPad1.0x1.5mm
- added C1: 100nF, Capacitor_SMD:C_0402_1005Metric_Pad0.74x0.62mm_HandSolder, F.Cu at (151.9, 103.6)
- added C27: 100nF, Capacitor_SMD:C_0402_1005Metric_Pad0.74x0.62mm_HandSolder, B.Cu at (137.1, 72.0)
- added C28: 100nF, Capacitor_SMD:C_0402_1005Metric_Pad0.74x0.62mm_HandSolder, B.Cu at (165.5, 94.8)
- added C29: 100nF, Capacitor_SMD:C_0402_1005Metric_Pad0.74x0.62mm_HandSolder, B.Cu at (145.6, 76.2)
- added C30: 100nF, Capacitor_SMD:C_0402_1005Metric_Pad0.74x0.62mm_HandSolder, B.Cu at (150.7, 72.0)
- added C31: 1uF, Capacitor_SMD:C_0603_1608Metric_Pad1.08x0.95mm_HandSolder, F.Cu at (135.3, 108.2)
- added C6: 100nF, Capacitor_SMD:C_0402_1005Metric_Pad0.74x0.62mm_HandSolder, F.Cu at (153.8, 94.1)
- added G***: LOGO, LogosZenith:Logo_29,1mm, F.Cu at (170.4, 116.0)
- added G***: LOGO, LOGO, B.Cu at (221.8, 96.8)
- added G***: LOGO, LogosZenith:Logo_29,1mm, B.Cu at (117.0, 116.3)
- added J1: BatBus, Connector_PinHeader_2.54mm:PinHeader_2x06_P2.54mm_Vertical, F.Cu at (139.2, 133.2)
- added R1: 10k, Resistor_SMD:R_0402_1005Metric_Pad0.72x0.64mm_HandSolder, F.Cu at (146.2, 105.5)
- added R11: *0R, Resistor_SMD:R_0402_1005Metric_Pad0.72x0.64mm_HandSolder, F.Cu at (124.3, 108.4)
- added R15: 10R, Resistor_SMD:R_0402_1005Metric_Pad0.72x0.64mm_HandSolder, B.Cu at (135.2, 72.6)
- added R16: 10R, Resistor_SMD:R_0402_1005Metric_Pad0.72x0.64mm_HandSolder, B.Cu at (135.2, 71.4)
- added R2: 10k, Resistor_SMD:R_0402_1005Metric_Pad0.72x0.64mm_HandSolder, F.Cu at (147.3, 105.5)
- added R21: 10R, Resistor_SMD:R_0402_1005Metric_Pad0.72x0.64mm_HandSolder, B.Cu at (146.2, 78.0)
- added R22: 10R, Resistor_SMD:R_0402_1005Metric_Pad0.72x0.64mm_HandSolder, B.Cu at (144.9, 78.0)
- added R23: 0R, Resistor_SMD:R_0402_1005Metric_Pad0.72x0.64mm_HandSolder, B.Cu at (142.5, 68.1)
- added R24: 10R, Resistor_SMD:R_0402_1005Metric_Pad0.72x0.64mm_HandSolder, B.Cu at (153.1, 70.7)
- added R25: 0R, Resistor_SMD:R_0402_1005Metric_Pad0.72x0.64mm_HandSolder, B.Cu at (144.5, 68.1)
- added R26: 0R, Resistor_SMD:R_0402_1005Metric_Pad0.72x0.64mm_HandSolder, B.Cu at (146.5, 68.1)
- added R27: 10R, Resistor_SMD:R_0402_1005Metric_Pad0.72x0.64mm_HandSolder, B.Cu at (153.1, 71.9)
- added R28: 0R, Resistor_SMD:R_0402_1005Metric_Pad0.72x0.64mm_HandSolder, B.Cu at (148.5, 68.1)
- added R3: 4k7, Resistor_SMD:R_0402_1005Metric_Pad0.72x0.64mm_HandSolder, F.Cu at (147.3, 86.2)
- added R4: 4k7, Resistor_SMD:R_0402_1005Metric_Pad0.72x0.64mm_HandSolder, F.Cu at (142.2, 85.2)
- added R7: *0R, Resistor_SMD:R_0402_1005Metric_Pad0.72x0.64mm_HandSolder, F.Cu at (124.3, 106.4)
- added U6: LM75B, Package_SO:VSSOP-8_3x3mm_P0.65mm, B.Cu at (165.6, 92.4)
- R30: renamed from R12; value R_Small -> 233k
- R33: renamed from R15; value R_Small -> 25,2k
- U2: value SN65HVD230 -> SN65HVD233
- moved JP2 25.0 mm to (131.1, 124.7), turned to 0 degrees
- moved U2 22.9 mm to (128.4, 97.0), turned to 180 degrees
- moved C4 21.3 mm to (132.8, 97.0), turned to 90 degrees
- moved JP1 13.3 mm to (116.2, 101.0)
- moved R30 2.75 mm to (136.2, 117.2)
- moved R32 2.75 mm to (134.9, 117.2)
- moved R33 2.75 mm to (136.2, 119.5)
- moved U8 2.75 mm to (131.4, 118.4)
- moved C25 2.58 mm to (155.6, 106.2)
- moved C32 2.58 mm to (138.6, 114.9)
- moved C33 2.58 mm to (145.3, 117.2)
- moved C34 2.58 mm to (159.3, 119.7)
- moved C35 2.58 mm to (139.1, 121.7)
- moved D4 2.58 mm to (143.3, 111.9)
- moved D5 2.58 mm to (146.6, 121.4)
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- renumbered C5 to C10, C6 to C11, C7 to C12, C8 to C13, C9 to C14, C10 to C15, C11 to C16, C12 to C17, C13 to C18, C14 to C19, C1 to C2, C15 to C20, C16 to C21, C17 to C22, C18 to C23, C19 to C24, C20 to C25, C21 to C26, C2 to C3, C22 to C32, C23 to C33, C24 to C34, C25 to C35, C3 to C4, C4 to C5, J1 to J2, J2 to J3, J3 to J4, J4 to J5, J5 to J6, R3 to R10, R4 to R12, R5 to R13, R6 to R14, R7 to R17, R8 to R18, R9 to R19, R10 to R20, R11 to R29, R13 to R31, R14 to R32, R16 to R34, R17 to R35, R1 to R8, R2 to R9, U6 to U7, U7 to U8, U8 to U9
Connections:
- net /Regulators/+3V3_PG renamed /+3V3_PG
- net /Regulators/+5V_PG renamed /+5V_PG
- C32 pad 1: -SOL_Sense -> SOL_Sense-
- D1 pad 1: +SOL_Sense -> SOL_Sense+
- D2 pad 1: +SOL_Sense -> SOL_Sense+
- D3 pad 1: +SOL_Sense -> SOL_Sense+
- D6 pad 1: +SOL_Sense -> SOL_Sense+
- J2 pad 16: BUS_CAN_H -> /BUS_CAN_H
- J2 pad 17: BUS_SDA -> /BUS_I2C_SDA
- J2 pad 18: BUS_CAN_L -> /BUS_CAN_L
- J2 pad 19: BUS_SCL -> /BUS_I2C_SCL
- J2 pad 8: SOL- -> GND
- JP2 pad 1: Net-(JP2-A) -> SOL_Sense-
- JP2 pad 2: +3.3VP -> /Charger/~{SHDN}
- R29 pad 1: +SOL_Sense -> SOL_Sense+
- R29 pad 2: -SOL_Sense -> SOL_Sense-
- R30 pad 2: -SOL_Sense -> SOL_Sense-
- U1 pad 14: unconnected-(U1-PA0-Pad14) -> /UART_Tx
- U1 pad 15: unconnected-(U1-PA1-Pad15) -> /UART_Rx
- U1 pad 29: unconnected-(U1-PB10-Pad29) -> /I2C2_SCL
- U1 pad 30: unconnected-(U1-PB11-Pad30) -> /I2C2_SDA
- U1 pad 38: unconnected-(U1-PC7-Pad38) -> /LBK
- U1 pad 44: unconnected-(U1-PA11-Pad44) -> /CAN_Rx
- U1 pad 45: unconnected-(U1-PA12-Pad45) -> /CAN_Tx
- U1 pad 58: unconnected-(U1-PB6-Pad58) -> /BUS_I2C_SCL
- U1 pad 59: unconnected-(U1-PB7-Pad59) -> /BUS_I2C_SDA
- U1 pad 60: unconnected-(U1-BOOT0-Pad60) -> /BOOT0
- U1 pad 7: unconnected-(U1-NRST-Pad7) -> /NRST
- U2 pad 5: unconnected-(U2-Vref-Pad5) -> /LBK
- U2 pad 6: unconnected-(U2-CANL-Pad6) -> /BUS_CAN_L
- U2 pad 7: unconnected-(U2-CANH-Pad7) -> /BUS_CAN_H
- U2 pad 8: unconnected-(U2-Rs-Pad8) -> GND
- U3 pad 3: /Regulators/+3V3_Enable -> /+3V3_En
- U4 pad 3: /Regulators/+5V_Enable -> /+5V_En
- U7 pad 1: +3V3 -> Net-(U7-IN-3)
- U7 pad 11: +5V -> Net-(U7-IN-1)
- U7 pad 12: +5V_Sense -> Net-(U7-IN+1)
- U7 pad 14: -SOL_Sense -> Net-(U7-IN-2)
- U7 pad 15: +SOL_Sense -> Net-(U7-IN+2)
- U7 pad 2: +3V3_Sense -> Net-(U7-IN+3)
- U7 pad 5: Net-(JP2-A) -> Net-(U7-A0)
- U7 pad 6: /Monitor/SCL -> /I2C2_SCL
- U7 pad 7: /Monitor/SDA -> /I2C2_SDA
- U8 pad 4: -SOL_Sense -> SOL_Sense-
- U9 pad 1: -SOL_Sense -> SOL_Sense-
- U9 pad 3: unconnected-(U8-~{SHDN}-Pad3) -> /Charger/~{SHDN}
Routing:
- net SOL_Sense+: track 0.00 -> 221.5 mm, vias 0 -> 18
- net SOL_Sense-: track 0.00 -> 61.3 mm, vias 0 -> 3
- net /I2C2_SDA: track 0.00 -> 44.7 mm, vias 0 -> 2
- net /I2C2_SCL: track 0.00 -> 40.2 mm, vias 0 -> 2
- net +3.3VP: track 23.6 -> 50.5 mm, vias 4 -> 14
- net Net-(U7-A0): track 0.00 -> 11.8 mm, vias 0 -> 1
- net GND: track 2.00 -> 11.8 mm, vias 111 -> 150
- net -SOL_Sense: track 9.21 -> 0.00 mm
- net +5V: track 17.3 -> 8.71 mm, vias 0 -> 1
- net Net-(U7-IN-1): track 0.00 -> 8.30 mm, vias 0 -> 1
- net Net-(U7-IN+1): track 0.00 -> 8.23 mm, vias 0 -> 1
- net +5V_Sense: track 29.7 -> 21.9 mm, vias 2 -> 3
- net Net-(D1-A): track 0.00 -> 6.25 mm
- net Net-(D6-A): track 0.00 -> 6.17 mm
- net Net-(U7-IN+3): track 0.00 -> 5.63 mm, vias 0 -> 1
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- added copper zone on F.Cu, net +3.3VP
- added copper zone on In2.Cu, net +3.3VP
- added copper zone on F.Cu, net +3V3
- added copper zone on F.Cu, net +5V
- added copper zone on In2.Cu, net BAT+
- added copper zone on In2.Cu, net GND
- added copper zone on F.Cu, net SOL_Sense+
- added copper zone on In2.Cu, net SOL_Sense+
- added copper zone on F.Cu, net SOL_Sense-
- removed copper zone on F.Cu, net -SOL_Sense
Other:
- outline, holes or cut-outs redrawn

Commit message: atualização esquema e pcb
Parts:
- added 16M1: Crystal_GND24, Crystal:Crystal_SMD_5032-4Pin_5.0x3.2mm, F.Cu at (160.2, 99.0)
- added C10: 7p, Capacitor_SMD:C_0402_1005Metric_Pad0.74x0.62mm_HandSolder, F.Cu at (176.7, 98.5)
- added C11: 7p, Capacitor_SMD:C_0402_1005Metric_Pad0.74x0.62mm_HandSolder, F.Cu at (176.7, 100.5)
- added C12: 33p, Capacitor_SMD:C_0402_1005Metric_Pad0.74x0.62mm_HandSolder, F.Cu at (118.9, 99.7)
- added C13: 4n7, Capacitor_SMD:C_0402_1005Metric_Pad0.74x0.62mm_HandSolder, F.Cu at (119.0, 97.1)
- added C14: 33p, Capacitor_SMD:C_0402_1005Metric_Pad0.74x0.62mm_HandSolder, F.Cu at (119.0, 94.8)
- added C7: 1u, Capacitor_SMD:C_0402_1005Metric_Pad0.74x0.62mm_HandSolder, F.Cu at (176.7, 92.6)
- added C8: 24p, Capacitor_SMD:C_0402_1005Metric_Pad0.74x0.62mm_HandSolder, F.Cu at (176.7, 94.6)
- added C9: 24p, Capacitor_SMD:C_0402_1005Metric_Pad0.74x0.62mm_HandSolder, F.Cu at (176.7, 96.6)
- added J3: Programmer, Connector_PinHeader_2.54mm:PinHeader_1x12_P2.54mm_Horizontal, F.Cu at (231.7, 46.1)
- added JP1: BOOT, Jumper:SolderJumper-3_P1.3mm_Open_RoundedPad1.0x1.5mm_NumberLabels, F.Cu at (177.2, 82.2)
- added R1: 10k, Resistor_SMD:R_0402_1005Metric_Pad0.72x0.64mm_HandSolder, F.Cu at (114.4, 114.1)
- added R14: 10k, Resistor_SMD:R_0402_1005Metric_Pad0.72x0.64mm_HandSolder, F.Cu at (121.5, 131.5)
- added R19: 10k, Resistor_SMD:R_0402_1005Metric_Pad0.72x0.64mm_HandSolder, F.Cu at (121.5, 129.5)
- added R2: 10k, Resistor_SMD:R_0402_1005Metric_Pad0.72x0.64mm_HandSolder, F.Cu at (114.4, 117.0)
- added R26: 0R, Resistor_SMD:R_0402_1005Metric_Pad0.72x0.64mm_HandSolder, F.Cu at (121.5, 113.6)
- added R28: 0R, Resistor_SMD:R_0402_1005Metric_Pad0.72x0.64mm_HandSolder, F.Cu at (121.5, 115.6)
- added R3: 390, Resistor_SMD:R_0402_1005Metric_Pad0.72x0.64mm_HandSolder, F.Cu at (114.4, 120.0)
- added R31: 0R, Resistor_SMD:R_0402_1005Metric_Pad0.72x0.64mm_HandSolder, F.Cu at (121.5, 117.6)
- added R34: 0R, Resistor_SMD:R_0402_1005Metric_Pad0.72x0.64mm_HandSolder, F.Cu at (121.5, 119.5)
- added R39: 0R, Resistor_SMD:R_0402_1005Metric_Pad0.72x0.64mm_HandSolder, F.Cu at (121.5, 123.5)
- added R41: 0R, Resistor_SMD:R_0402_1005Metric_Pad0.72x0.64mm_HandSolder, F.Cu at (121.5, 125.5)
- added R8: 60, Resistor_SMD:R_0603_1608Metric_Pad0.98x0.95mm_HandSolder, F.Cu at (122.0, 98.2)
- added R9: 60, Resistor_SMD:R_0603_1608Metric_Pad0.98x0.95mm_HandSolder, F.Cu at (122.0, 95.9)
- added S1: RST, Button_Switch_SMD:SW_Push_1P1T_NO_CK_KMR2, F.Cu at (218.7, 70.2)
- added Y1: 32,768k, Crystal:Crystal_SMD_3215-2Pin_3.2x1.5mm, F.Cu at (166.1, 100.2)
- JP2: renamed from JP1; moved to B.Cu
- U6: footprint Package_SO:VSSOP-8_3x3mm_P0.65mm -> Package_SO:Texas_S-PDSO-G8_3x3mm_P0.65mm
- moved JP2 49.1 mm to (152.7, 68.2), turned to 180 degrees
- renumbered C10 to C15, C11 to C16, C12 to C17, C13 to C18, C14 to C19, C15 to C20, C16 to C21, C17 to C22, C18 to C23, C19 to C24, C20 to C25, C21 to C26, C22 to C27, C23 to C28, C24 to C29, C25 to C30, C26 to C31, C27 to C32, C28 to C33, C29 to C34, C30 to C35, C31 to C36, C32 to C37, C33 to C38, C34 to C39, C35 to C40, J3 to J4, J4 to J5, J5 to J6, J6 to J7, R7 to R10, R8 to R11, R9 to R12, R10 to R13, R11 to R15, R12 to R16, R13 to R17, R14 to R18, R15 to R20, R16 to R21, R17 to R22, R18 to R23, R19 to R24, R20 to R25, R21 to R27, R22 to R29, R23 to R30, R24 to R32, R25 to R33, R26 to R35, R27 to R36, R28 to R37, R29 to R38, R1 to R4, R30 to R40, R31 to R42, R32 to R43, R33 to R44, R34 to R45, R35 to R46, R2 to R5, R3 to R6, R4 to R7
Connections:
- J2 pad 13: BUS_MISO -> unconnected-(J2-Pin_13-Pad13)
- J2 pad 14: BUS_MOSI -> unconnected-(J2-Pin_14-Pad14)
- J2 pad 15: BUS_SCLK -> unconnected-(J2-Pin_15-Pad15)
- J2 pad 7: SOL+ -> SOL_Sense-
- U1 pad 21: unconnected-(U1-PA5-Pad21) -> /SPI1_SCK
- U1 pad 22: unconnected-(U1-PA6-Pad22) -> /SPI1_MISO
- U1 pad 23: unconnected-(U1-PA7-Pad23) -> /SPI1_MOSI
- U1 pad 3: unconnected-(U1-PC14-Pad3) -> /OSC32_IN
- U1 pad 4: unconnected-(U1-PC15-Pad4) -> /OSC32_OUT
- U1 pad 46: unconnected-(U1-PA13-Pad46) -> /SWDIO
- U1 pad 49: unconnected-(U1-PA14-Pad49) -> /SWCLK
- U1 pad 5: unconnected-(U1-PH0-Pad5) -> /OSC_IN
- U1 pad 55: unconnected-(U1-PB3-Pad55) -> /SWO
- U1 pad 6: unconnected-(U1-PH1-Pad6) -> /OSC_OUT
- U6 pad 6: GND -> Net-(U6-A1)
- U6 pad 7: GND -> Net-(U6-A0)
- U9 pad 3: /Charger/~{SHDN} -> Net-(U9-~{SHDN})
- U9 pad 8: /Charger/NTC -> /NTC
Routing:
- net Net-(JP2-A): track 2.57 -> 12.3 mm
- net +3.3VP: track 50.5 -> 53.5 mm
- net /NTC: track 0.00 -> 1.92 mm, vias 0 -> 1
- net /Charger/NTC: track 1.92 -> 0.00 mm, vias 1 -> 0
- net Net-(U9-~{SHDN}): track 0.00 -> 1.72 mm, vias 0 -> 1
- net /Charger/~{SHDN}: track 3.63 -> 1.91 mm, vias 2 -> 1
