File: Main Board/Kicad/Power Supply ZensatV3.kicad_pcb (KiCad board)
At the start: 4 copper layers, 86 x 86 mm, 120 parts, among them J1 BatBus, J2 ZenBus, J3 Programmer, J4 Conn_01x02_Pin, J5 Conn_01x02_Pin, J6 Conn_01x02_Pin, J7 Conn_01x02_Pin, U1 STM32L476RGTx, U2 SN65HVD233, U3 LMR33630ADDA, U4 LMR33630ADDA, U5 AMS1117-3.3, U6 LM75B, U7 INA3221, U8 LM234DT, U9 LT3652IMSE, Y1 32,768k

Commit message: atualização
Parts:
- removed 16M1: Crystal_GND24, Crystal:Crystal_SMD_5032-4Pin_5.0x3.2mm
- removed C8, C9: 24p, Capacitor_SMD:C_0402_1005Metric_Pad0.74x0.62mm_HandSolder
- removed the G*** at (221.8, 96.8)
- removed JP2 (x2): SolderJumper_2_Open, Jumper:SolderJumper-2_P1.3mm_Open_RoundedPad1.0x1.5mm
- removed R10, R15: *0R, Resistor_SMD:R_0402_1005Metric_Pad0.72x0.64mm_HandSolder
- removed R3: 390, Resistor_SMD:R_0402_1005Metric_Pad0.72x0.64mm_HandSolder
- added G***: LOGO, LOGO, F.Cu at (122.5, 120.8)
- added G***: LOGO, LOGO, F.Cu at (115.5, 115.6)
- added G***: LOGO, LOGO, F.Cu at (123.0, 110.4)
- added G***: LOGO, LOGO, B.Cu at (176.3, 94.2)
- added G***: LOGO, LOGO, B.Cu at (170.2, 119.7)
- C10, C11, R26, R28, R31, R34, Y1: moved to B.Cu
- J3: footprint Connector_PinHeader_2.54mm:PinHeader_1x12_P2.54mm_Horizontal -> Connector_Hirose:Hirose_DF13-12P-1.25DSA_1x12_P1.25mm_Vertical
- moved J3 69.3 mm to (182.7, 95.0), turned to -90 degrees
- moved R2 62.4 mm to (171.9, 92.8)
- moved R14 56.6 mm to (156.3, 86.8)
- moved R1 47.4 mm to (159.1, 98.2), turned to 90 degrees
- moved R34 46.4 mm to (162.9, 98.6)
- moved R31 46.1 mm to (162.9, 97.5)
- moved R28 45.7 mm to (162.9, 96.4)
- moved R26 45.3 mm to (162.9, 95.3)
- moved S1 45.3 mm to (177.2, 88.5), turned to -90 degrees
- moved R19 38.7 mm to (131.1, 92.0)
- moved C10 20.5 mm to (156.3, 101.0), turned to 90 degrees
- moved C11 20.5 mm to (156.3, 98.1), turned to 90 degrees
- moved C7 19.9 mm to (157.6, 98.2), turned to -90 degrees
- moved Y1 11.7 mm to (154.4, 99.5), turned to 90 degrees
- moved R41 10.7 mm to (131.9, 123.2), turned to 180 degrees
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Connections:
- net /BUS_CAN_H renamed /BUS_CAN+
- net /BUS_CAN_L renamed /BUS_CAN-
- J2 pad 7: SOL_Sense- -> SOL_Sense+
- J3 pad 1: +3V3 -> +3.3VP
- JP1 pad 3: +3V3 -> +3.3VP
- R1 pad 1: +3V3 -> +3.3VP
- R22 pad 2: Net-(JP2-A) -> +3.3VP
- U1 pad 5: /OSC_IN -> unconnected-(U1-PH0-Pad5)
- U1 pad 6: /OSC_OUT -> unconnected-(U1-PH1-Pad6)
- U7 pad 16: Net-(JP2-A) -> +3.3VP
Routing:
- net +3.3VP: track 53.5 -> 134.6 mm, vias 14 -> 23
- net /BUS_CAN-: track 0.00 -> 76.1 mm, vias 0 -> 1
- net /BUS_CAN+: track 0.00 -> 75.5 mm, vias 0 -> 1
- net /BOOT0: track 0.00 -> 51.0 mm, vias 0 -> 1
- net /SWDIO: track 0.00 -> 50.9 mm, vias 0 -> 2
- net /SWCLK: track 0.00 -> 50.6 mm, vias 0 -> 2
- net /NRST: track 0.00 -> 47.9 mm, vias 0 -> 2
- net /SWO: track 0.00 -> 42.2 mm, vias 0 -> 2
- net /Charger/~{SHDN}: track 1.91 -> 35.8 mm, vias 1 -> 0
- net /UART_Tx: track 0.00 -> 33.3 mm
- net /UART_Rx: track 0.00 -> 33.0 mm
- net GND: track 11.8 -> 38.4 mm, vias 150 -> 175
- net SOL_Sense+: track 221.5 -> 239.5 mm
- net /NTC: track 1.92 -> 16.6 mm
- net /LBK: track 0.00 -> 14.7 mm
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
Commit message: atualização pcb/esquema
Parts:
- added C41: 220nF, Capacitor_SMD:C_0402_1005Metric_Pad0.74x0.62mm_HandSolder, F.Cu at (125.2, 83.0)
- added C42: 220nF, Capacitor_SMD:C_0402_1005Metric_Pad0.74x0.62mm_HandSolder, F.Cu at (160.3, 83.0)
- added D7: LED, LED_SMD:LED_0805_2012Metric_Pad1.15x1.40mm_HandSolder, F.Cu at (176.9, 67.0)
- added D8: LED, LED_SMD:LED_0805_2012Metric_Pad1.15x1.40mm_HandSolder, F.Cu at (176.9, 70.1)
- added G***: LOGO, LOGO, F.Cu at (174.9, 114.4)
- added R10: 10k, Resistor_SMD:R_0402_1005Metric_Pad0.72x0.64mm_HandSolder, F.Cu at (138.9, 103.4)
- added R15: 1k, Resistor_SMD:R_0402_1005Metric_Pad0.72x0.64mm_HandSolder, F.Cu at (149.7, 85.5)
- added R47: 1k, Resistor_SMD:R_0402_1005Metric_Pad0.72x0.64mm_HandSolder, F.Cu at (134.6, 93.0)
- added R48: 10k, Resistor_SMD:R_0402_1005Metric_Pad0.72x0.64mm_HandSolder, F.Cu at (137.6, 103.4)
- C29: value 100nF -> 100nF 25V
- C30: value 10uF -> 10uF 10V
- C31, C32, C34, C35: value 100nF -> 100nF 10V
- C39: value 10uF -> 10uF 25V
- moved R41 9.28 mm to (127.5, 115.0), turned to -90 degrees
- moved R14 6.60 mm to (149.7, 87.0)
- moved R19 3.54 mm to (134.6, 91.5)
- moved G*** 1.41 mm to (168.9, 115.8)
- moved C23 1.15 mm to (122.2, 83.8)
- moved C16 0.95 mm to (157.3, 83.8)
- moved C38 0.77 mm to (146.1, 117.0)
- moved C36 0.43 mm to (135.3, 108.6)
Connections:
- J2 pad 34: unconnected-(J2-Pin_34-Pad34) -> /~{CHRG}
- R22 pad 1: /Monitor/PV -> /PV
- R23 pad 1: /Monitor/CRITICAL -> /CRITICAL
- R24 pad 1: /Monitor/WARNING -> /WARNING
- R25 pad 1: /Monitor/TC -> /TC
- R41 pad 1: /Charger/~{SHDN} -> /~{SHDN}
- U1 pad 17: unconnected-(U1-PA3-Pad17) -> /+3V3_PG
- U1 pad 20: unconnected-(U1-PA4-Pad20) -> /+3V3_En
- U1 pad 25: unconnected-(U1-PC5-Pad25) -> /PV
- U1 pad 26: unconnected-(U1-PB0-Pad26) -> /CRITICAL
- U1 pad 27: unconnected-(U1-PB1-Pad27) -> /WARNING
- U1 pad 28: unconnected-(U1-PB2-Pad28) -> /TC
- U1 pad 36: unconnected-(U1-PB15-Pad36) -> /+5V_PG
- U1 pad 37: unconnected-(U1-PC6-Pad37) -> /+5V_En
- U1 pad 50: unconnected-(U1-PA15-Pad50) -> /~{CHRG}
- U1 pad 51: unconnected-(U1-PC10-Pad51) -> /~{FAULT}
- U1 pad 52: unconnected-(U1-PC11-Pad52) -> /~{SHDN}
- U3 pad 3: /+3V3_En -> Net-(U3-EN)
- U4 pad 3: /+5V_En -> Net-(U4-EN)
- U7 pad 10: /Monitor/PV -> /PV
- U7 pad 13: /Monitor/TC -> /TC
- U7 pad 8: /Monitor/WARNING -> /WARNING
- U7 pad 9: /Monitor/CRITICAL -> /CRITICAL
- U9 pad 4: /Charger/~{CHRG} -> /~{CHRG}
- U9 pad 5: /Charger/~{FAULT} -> /~{FAULT}
Routing:
- net /BUS_I2C_SDA: track 4.88 -> 98.7 mm, vias 1 -> 3
- net /BUS_I2C_SCL: track 4.88 -> 97.4 mm, vias 1 -> 3
- net /I2C2_SCL: track 43.8 -> 131.8 mm, vias 2 -> 4
- net /I2C2_SDA: track 48.0 -> 132.7 mm, vias 2 -> 4
- net BAT+: track 4.93 -> 75.2 mm, vias 31 -> 34
- net /Charger/~{SHDN}: track 35.8 -> 0.00 mm
- net /WARNING: track 0.00 -> 31.0 mm, vias 0 -> 2
- net /CRITICAL: track 0.00 -> 29.8 mm, vias 0 -> 2
- net /~{FAULT}: track 0.00 -> 27.4 mm, vias 0 -> 2
- net /PV: track 0.00 -> 27.2 mm, vias 0 -> 2
- net /~{CHRG}: track 0.00 -> 26.2 mm, vias 0 -> 2
- net /~{SHDN}: track 0.00 -> 26.1 mm
- net /TC: track 0.00 -> 22.1 mm
- net /+3V3_PG: track 1.72 -> 21.5 mm, vias 1 -> 0
- net /+5V_PG: track 1.69 -> 17.9 mm, vias 1 -> 0
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
Commit message: atualização
Parts:
- added REF**: ESD-Logo_6.6x6mm_SilkScreen, Symbol:ESD-Logo_6.6x6mm_SilkScreen, F.Cu at (168.9, 97.4)
- added REF**: KiCad-Logo2_6mm_SilkScreen, Symbol:KiCad-Logo2_6mm_SilkScreen, B.Cu at (116.9, 76.4)
- moved D8 7.54 mm to (176.8, 77.6)
- moved D7 7.18 mm to (176.8, 74.2)
Other:
- board text added: "CAN"
- board text added: "Monitor"

Commit message: Main Board V1.0
Conclusão da Main Board.
Parts:
- removed the REF** at (168.9, 97.4)
- added D9: LEDR, LED_SMD:LED_0805_2012Metric_Pad1.15x1.40mm_HandSolder, F.Cu at (178.3, 111.1)
- added J8: External Power, Connector_Molex:Molex_PicoBlade_53261-0671_1x06-1MP_P1.25mm_Horizontal, F.Cu at (182.4, 100.6)
- added R49: 470R, Resistor_SMD:R_0402_1005Metric_Pad0.72x0.64mm_HandSolder, F.Cu at (175.6, 73.6)
- added R50: 470R, Resistor_SMD:R_0402_1005Metric_Pad0.72x0.64mm_HandSolder, F.Cu at (141.7, 83.7)
- added R51: 10k, Resistor_SMD:R_0402_1005Metric_Pad0.72x0.64mm_HandSolder, F.Cu at (178.3, 107.4)
- added REF**: Symbol_HighVoltage_Triangle_8x7mm_Copper, Symbol:Symbol_HighVoltage_Triangle_8x7mm_Copper, F.Cu at (122.0, 126.5)
- D7, D8: value LED -> LEDG
- J3: footprint Connector_Hirose:Hirose_DF13-12P-1.25DSA_1x12_P1.25mm_Vertical -> Connector_Molex:Molex_PicoBlade_53261-1071_1x10-1MP_P1.25mm_Horizontal; moved to B.Cu
- moved D8 37.5 mm to (139.8, 84.4), turned to 90 degrees
- moved G*** 6.54 mm to (176.0, 87.7)
- moved J3 5.55 mm to (182.4, 100.6)
- moved D7 3.00 mm to (175.2, 76.8), turned to 90 degrees
- moved G*** 2.11 mm to (122.3, 118.7)
- moved G*** 1.01 mm to (122.5, 109.5)
- moved G*** 1.00 mm to (115.5, 116.6)
- moved R47 0.10 mm to (134.6, 92.9)
Connections:
- net SOL_Sense+ renamed SOL+
- D7 pad 2: unconnected-(D7-A-Pad2) -> Net-(D7-A)
- D8 pad 2: unconnected-(D8-A-Pad2) -> Net-(D8-A)
- J2 pad 13: unconnected-(J2-Pin_13-Pad13) -> /SPI1_MISO
- J2 pad 14: unconnected-(J2-Pin_14-Pad14) -> /SPI1_MOSI
- J2 pad 15: unconnected-(J2-Pin_15-Pad15) -> /SPI1_SCK
- J2 pad 34: /~{CHRG} -> unconnected-(J2-Pin_34-Pad34)
- U1 pad 1: unconnected-(U1-VBAT-Pad1) -> +3.3VP
- U1 pad 34: unconnected-(U1-PB13-Pad34) -> /Heater
- U1 pad 35: unconnected-(U1-PB14-Pad35) -> /Deploy
- U1 pad 9: unconnected-(U1-PC1-Pad9) -> /DebugLed
Routing:
- net +3.3VP: track 127.2 -> 207.4 mm, vias 27 -> 32
- net /Heater: track 0.00 -> 45.8 mm, vias 0 -> 1
- net /SPI1_MOSI: track 0.00 -> 45.0 mm, vias 0 -> 1
- net /Deploy: track 0.00 -> 39.7 mm, vias 0 -> 1
- net /SPI1_SCK: track 0.00 -> 38.1 mm, vias 0 -> 1
- net /DebugLed: track 0.00 -> 37.6 mm
- net /SPI1_MISO: track 0.00 -> 36.1 mm, vias 0 -> 2
- net BAT+: track 75.2 -> 105.8 mm, vias 34 -> 35
- net /+3V3_PG: track 21.5 -> 48.0 mm
- net /+5V_PG: track 17.9 -> 27.5 mm
- net SOL+: track 240.4 -> 245.0 mm, vias 18 -> 19
- net GND: track 36.8 -> 40.6 mm, vias 228 -> 229
- net Net-(D7-A): track 0.00 -> 2.30 mm
- net /UART_Rx: track 33.0 -> 30.8 mm, vias 0 -> 1
- net /NRST: track 47.9 -> 45.8 mm
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Other:
- board text added: "08/10/2026"
