File: Main Board/Kicad/charger.kicad_sch (KiCad schematic)
At the start: 12 parts, among them U8 LT3652IMSE

Commit message: Atualização do circuito/pcb
Parts:
- removed D5: D_Schottky, symbol Device:D_Schottky
- added C19: 10uF, Capacitor_SMD:C_1206_3216Metric_Pad1.33x1.80mm_HandSolder, symbol Device:C_Small
- added C20: 680nF, Capacitor_SMD:C_0402_1005Metric_Pad0.74x0.62mm_HandSolder, symbol Device:C_Small
- added D4: MBRS340, Diode_SMD:D_SMC, symbol Diode:MBRS340
- added D6: 1N5819HW, Diode_SMD:D_SOD-123, symbol Device:D_Schottky
- added R11: 626k, Resistor_SMD:R_0402_1005Metric_Pad0.72x0.64mm_HandSolder, symbol Device:R_Small
- added R12: 412k, Resistor_SMD:R_0402_1005Metric_Pad0.72x0.64mm_HandSolder, symbol Device:R_Small
- added R9: 1k, Resistor_SMD:R_0402_1005Metric_Pad0.72x0.64mm_HandSolder, symbol Device:R_Small
- added U8: LM234DT, Package_SO:SOIC-8_3.9x4.9mm_P1.27mm, symbol Reference_Current:LM234Z-3
- C17: footprint (none) -> Capacitor_SMD:C_1206_3216Metric_Pad1.33x1.80mm_HandSolder
- C18: value C_Small -> 1uF; footprint (none) -> Capacitor_SMD:C_0402_1005Metric_Pad0.74x0.62mm_HandSolder
- D1, D2, D3: value D_Schottky -> 1N5819HW; footprint (none) -> Diode_SMD:D_SOD-123
- D5: renamed from D4; value D_Schottky -> 1N5819HW; footprint (none) -> Diode_SMD:D_SOD-123
- L3: value L -> 47uH; footprint (none) -> Inductor_SMD:L_TDK_SLF7032
- R10: renamed from R8; footprint (none) -> Resistor_SMD:R_0402_1005Metric_Pad0.72x0.64mm_HandSolder
- R7: footprint (none) -> Resistor_SMD:R_0402_1005Metric_Pad0.72x0.64mm_HandSolder
- R8: renamed from R9; value R_Small -> 0R33; footprint (none) -> Resistor_SMD:R_1210_3225Metric_Pad1.30x2.65mm_HandSolder
- renumbered U8 to U9
Connections:
- net GND: now also C19.2, C20.2, D4.2 (A), R12.1; no longer U9.6 (TIMER)
- net at C17.1, D1.1 (K), D2.1 (K)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: now also U9.3 (~{SHDN}), U8.4
- net SOL4: now reaches D5.2 (A)
- net at R10.2, R7.1, U9.2 (V_{IN_REG}): now also R9.1, U8.6
- net +BATT: now reaches R8.2, U9.9 (BAT)
- net +BATT: now also C19.1, D6.2 (A), R11.2
- net SOL3: now reaches D3.2 (A)
- net at C18.2, U9.11 (BOOST): now also D6.1 (K)
- net at C18.1, L3.1, U9.12 (SW): now also D4.1 (K)
- net ~{CHRG}: now reaches U9.4 (~{CHRG})
- net ~{FAULT}: now reaches U9.5 (~{FAULT})
- net at U9.7 (V_{FB}): now also R11.1, R12.2
- net NTC: now reaches U9.8 (NTC)
- net SOL1: now reaches D1.2 (A)
- net SOL2: now reaches D2.2 (A)
- new net: R9.2, U8.1
- new net: C20.1, U9.6 (TIMER)
Other:
- moved on the sheet: C17, C18, D1, D2, D3, D5, L3, R10, R7, R8, U9

Commit message: atualização pcb
Parts:
- added J2, J3, J4, J5: Conn_01x02_Pin, Connector_JST:JST_ZH_B2B-ZR_1x02_P1.50mm_Vertical, symbol Connector:Conn_01x02_Pin
- added JP6: SolderJumper_2_Open, Jumper:SolderJumper-2_P1.3mm_Open_RoundedPad1.0x1.5mm, symbol Jumper:SolderJumper_2_Open
- added R11: 0R33, Resistor_SMD:R_1210_3225Metric_Pad1.30x2.65mm_HandSolder, symbol Device:R_Small
- C22: renamed from C17; footprint Capacitor_SMD:C_1206_3216Metric_Pad1.33x1.80mm_HandSolder -> Capacitor_SMD:C_0805_2012Metric_Pad1.18x1.45mm_HandSolder
- C23: renamed from C18; value 1uF -> 1uF 50V; footprint Capacitor_SMD:C_0402_1005Metric_Pad0.74x0.62mm_HandSolder -> Capacitor_SMD:C_0603_1608Metric_Pad1.08x0.95mm_HandSolder
- D4: value MBRS340 -> SS34; footprint Diode_SMD:D_SMC -> Diode_SMD:D_SMA
- renumbered C19 to C24, C20 to C25, D6 to D5, D5 to D6, R7 to R12, R8 to R13, R9 to R14, R10 to R15, R11 to R16, R12 to R17, U8 to U7, U9 to U8
Connections:
- net GND: now also J2.2 (Pin_2), J3.2 (Pin_2), J4.2 (Pin_2), J5.2 (Pin_2)
- net SOL1: no longer names the net of D1.2 (A)
- net SOL1: now also J2.1 (Pin_1)
- net SOL2: no longer names the net of D2.2 (A)
- net SOL2: now also J3.1 (Pin_1)
- net SOL3: no longer names the net of D3.2 (A)
- net SOL3: now also J4.1 (Pin_1)
- net SOL4: no longer names the net of D6.2 (A)
- net SOL4: now also J5.1 (Pin_1)
- new net +SOL_Sense: D1.1 (K), D2.1 (K), D3.1 (K), D6.1 (K), R11.1
- new net -SOL_Sense: C22.1, JP6.1 (A), R11.2, R12.2, U7.4, U8.1 (V_{IN})
- new net ~{SHDN}: JP6.2 (B), U8.3 (~{SHDN})
Other:
- note added: "Solar MPPT & Battery charger"
- moved on the sheet: C22, C23, C24, C25, D1, D2, D3, D4, D5, D6, L3, R12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

Commit message: atualização pcb
Parts:
- added C31: 1uF, Capacitor_SMD:C_0603_1608Metric_Pad1.08x0.95mm_HandSolder, symbol Device:C_Small
- R30: renamed from R12; value R_Small -> 233k
- R33: renamed from R15; value R_Small -> 25,2k
- renumbered C22 to C32, C23 to C33, C24 to C34, C25 to C35, J2 to J3, J3 to J4, J4 to J5, J5 to J6, JP6 to JP2, R11 to R29, R13 to R31, R14 to R32, R16 to R34, R17 to R35, U7 to U8, U8 to U9
Connections:
- net GND: now also C31.1
- net +SOL_Sense renamed SOL_Sense+
- net SOL_Sense+: now also C31.2
- net -SOL_Sense renamed SOL_Sense-

Commit message: atualização esquema e pcb
Parts:
- removed JP2: SolderJumper_2_Open, Jumper:SolderJumper-2_P1.3mm_Open_RoundedPad1.0x1.5mm, symbol Jumper:SolderJumper_2_Open
- added R39, R41: 0R, Resistor_SMD:R_0402_1005Metric_Pad0.72x0.64mm_HandSolder, symbol Device:R_Small
- renumbered C31 to C36, C32 to C37, C33 to C38, C34 to C39, C35 to C40, J3 to J4, J4 to J5, J5 to J6, J6 to J7, R29 to R38, R30 to R40, R31 to R42, R32 to R43, R33 to R44, R34 to R45, R35 to R46
Connections:
- net SOL_Sense-: now also R39.2
- net ~{SHDN}: now also R41.1; no longer U9.3 (~{SHDN})
- new net: R39.1, R41.2, U9.3 (~{SHDN})

Commit message: atualização pcb/esquema
Parts:
- C39: value 10uF -> 10uF 25V
Changed lines of the file:
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@@
 			)
 		)
-		(property "Value" "10uF"
+		(property "Value" "10uF 25V"
 			(at 232.41 99.0662 0)
 			(show_name no)

Commit message: Main Board V1.0
Conclusão da Main Board.
Connections:
- net SOL_Sense+ renamed SOL+
Changed lines of the file:
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@@
 	)
 	(junction
+		(at 156.21 82.55)
+		(diameter 0)
+		(color 0 0 0 0)
+	)
+	(junction
 		(at 99.06 82.55)
 		(diameter 0)
@@
 	(wire
 		(pts
+			(xy 156.21 81.28) (xy 156.21 82.55)
+		)
+		(stroke
+			(width 0)
+			(type default)
+		)
+	)
+	(wire
+		(pts
 			(xy 50.8 91.44) (xy 52.07 91.44)
 		)
@@
 		)
 	)
-	(global_label "SOL_Sense+"
+	(global_label "SOL+"
 		(shape input)
 		(at 77.47 78.74 90)
@@
 		)
 		(property "Intersheetrefs" "${INTERSHEET_REFS}"
-			(at 77.47 64.0829 90)
+			(at 77.47 70.6143 90)
 			(hide yes)
 			(show_name no)
@@
 					(unit 1)
 				)
+			)
+		)
+	)
+	(symbol
+		(lib_id "power:PWR_FLAG")
+		(at 156.21 81.28 0)
+		(unit 1)
+		(body_style 1)
+		(exclude_from_sim no)
+		(in_bom yes)
+		(on_board yes)
+		(in_pos_files yes)
+		(dnp no)
+		(fields_autoplaced yes)
+		(property "Reference" "#FLG02"
+			(at 156.21 79.375 0)
+			(hide yes)
+			(show_name no)
+			(do_not_autoplace no)
+			(effects
+				(font
+					(size 1.27 1.27)
+				)
+			)
+		)
+		(property "Value" "PWR_FLAG"
+			(at 156.21 76.2 0)
+			(show_name no)
+			(do_not_autoplace no)
+			(effects
+				(font
+					(size 1.27 1.27)
+				)
+			)
+		)
+		(property "Footprint" ""
+			(at 156.21 81.28 0)
+			(hide yes)
+			(show_name no)
+			(do_not_autoplace no)
+			(effects
+				(font
+					(size 1.27 1.27)
+				)
+			)
+		)
+		(property "Datasheet" ""
+			(at 156.21 81.28 0)
+			(hide yes)
+			(show_name no)
+			(do_not_autoplace no)
+			(effects
+				(font
+					(size 1.27 1.27)
+				)
+			)
+		)
+		(property "Description" "Special symbol for telling ERC where power comes from"
+			(at 156.21 81.28 0)
+			(hide yes)
+			(show_name no)
+			(do_not_autoplace no)
+			(effects
+				(font
+					(size 1.27 1.27)
+				)
+			)
+		)
+		(pin "1"
+		)
+		(instances
+			(project "Power Supply ZensatV3"
+				(path "/64de738a-78a3-405a-9208-2090dc1f201b/2e922904-ff10-4af4-b918-0c7939a35aa2"
+					(reference "#FLG02")
+					(unit 1)
+				)
