File: Main Board/Kicad/main.kicad_sch (KiCad schematic)
At the start: 2 parts, among them J1 ZenBus, U1 STM32L476RGTx

Commit message: Atualização do circuito/pcb
Other:
- sheet Charger ports: added NTC, SOL1, SOL2, SOL3, SOL4, ~{CHRG}, ~{FAULT}; removed none
Changed lines of the file:
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@@
+	)
+	(no_connect
+		(at 264.16 55.88)
 	)
 	(no_connect
@@
 	)
 	(no_connect
-		(at 264.16 55.88)
-	)
-	(no_connect
 		(at 264.16 73.66)
 	)
 	(no_connect
+		(at 264.16 50.8)
+	)
+	(no_connect
+		(at 264.16 48.26)
+	)
+	(no_connect
 		(at 264.16 58.42)
-	)
-	(no_connect
-		(at 264.16 50.8)
-	)
-	(no_connect
-		(at 264.16 48.26)
 	)
 	(no_connect
@@
 		(dnp no)
 		(fields_autoplaced yes)
-		(property "Reference" "#PWR01"
+		(property "Reference" "#PWR05"
 			(at 63.5 153.67 0)
 			(hide yes)
@@
 			(project "Power Supply ZensatV3"
 				(path "/64de738a-78a3-405a-9208-2090dc1f201b"
-					(reference "#PWR01")
+					(reference "#PWR05")
 					(unit 1)
 				)
@@
 		(dnp no)
 		(fields_autoplaced yes)
-		(property "Reference" "#PWR013"
+		(property "Reference" "#PWR01"
 			(at 168.91 24.13 0)
 			(hide yes)
@@
 			(project "Power Supply ZensatV3"
 				(path "/64de738a-78a3-405a-9208-2090dc1f201b"
-					(reference "#PWR013")
+					(reference "#PWR01")
 					(unit 1)
 				)
@@
 		(dnp no)
 		(fields_autoplaced yes)
-		(property "Reference" "#PWR015"
+		(property "Reference" "#PWR04"
 			(at 168.91 39.37 0)
 			(hide yes)
@@
 			(project "Power Supply ZensatV3"
 				(path "/64de738a-78a3-405a-9208-2090dc1f201b"
-					(reference "#PWR015")
+					(reference "#PWR04")
 					(unit 1)
 				)
@@
 		(dnp no)
 		(fields_autoplaced yes)
-		(property "Reference" "#PWR014"
+		(property "Reference" "#PWR02"
 			(at 175.26 24.13 0)
 			(hide yes)
@@
 			(project "Power Supply ZensatV3"
 				(path "/64de738a-78a3-405a-9208-2090dc1f201b"
-					(reference "#PWR014")
+					(reference "#PWR02")
 					(unit 1)
 				)
@@
 		(dnp no)
 		(fields_autoplaced yes)
-		(property "Reference" "#PWR019"
+		(property "Reference" "#PWR03"
 			(at 181.61 24.13 0)
 			(hide yes)
@@
 			(project "Power Supply ZensatV3"
 				(path "/64de738a-78a3-405a-9208-2090dc1f201b"
-					(reference "#PWR019")
+					(reference "#PWR03")
 					(unit 1)
 				)
@@
 	)
 	(sheet
-		(at 173.99 99.06)
-		(size 25.4 36.83)
+		(at 173.99 80.01)
+		(size 20.32 24.13)
 		(exclude_from_sim no)
 		(in_bom yes)
@@
 		)
 		(property "Sheetname" "Charger"
-			(at 173.99 98.3484 0)
+			(at 173.99 79.2984 0)
 			(show_name no)
 			(do_not_autoplace no)
@@
 		)
 		(property "Sheetfile" "charger.kicad_sch"
-			(at 173.99 136.4746 0)
+			(at 173.99 104.7246 0)
 			(show_name no)
 			(do_not_autoplace no)
@@
 			)
 		)
+		(pin "NTC" passive
+			(at 173.99 82.55 180)
+			(effects
+				(font
+					(size 1.27 1.27)
+				)
+				(justify left)
+			)
+		)
+		(pin "SOL1" input
+			(at 173.99 86.36 180)
+			(effects
+				(font
+					(size 1.27 1.27)
+				)
+				(justify left)
+			)
+		)
+		(pin "SOL2" input
+			(at 173.99 88.9 180)
+			(effects
+				(font
+					(size 1.27 1.27)
+				)
+				(justify left)
+			)
+		)
+		(pin "SOL3" input
+			(at 173.99 91.44 180)
+			(effects
+				(font
+					(size 1.27 1.27)
+				)
+				(justify left)
+			)
+		)
+		(pin "SOL4" input
+			(at 173.99 93.98 180)
+			(effects
+				(font
+					(size 1.27 1.27)
+				)
+				(justify left)
+			)
+		)
+		(pin "~{CHRG}" output
+			(at 173.99 97.79 180)
+			(effects
+				(font
+					(size 1.27 1.27)
+				)
+				(justify left)
+			)
+		)
+		(pin "~{FAULT}" output
+			(at 173.99 101.6 180)
+			(effects
+				(font
+					(size 1.27 1.27)
+				)
+				(justify left)
+			)
+		)

Commit message: atualização pcb
Parts:
- added C1, C2, C26, C3, C4: 100nF, Capacitor_SMD:C_0402_1005Metric_Pad0.74x0.62mm_HandSolder, symbol Device:C_Small
- added U2: SN65HVD230, Package_SO:SOIC-8_3.9x4.9mm_P1.27mm, symbol Interface_CAN_LIN:SN65HVD230
Connections:
- net GND: now also C1.1, C2.1, C26.1, C3.1, C4.1, U2.2 (GND)
- net +3.3VP: now reaches U1.13 (VDDA)
- net +3.3VP: now also U1.19 (VDD), U1.32 (VDD), U1.48 (VDDUSB), U1.64 (VDD), C1.2, C2.2, C26.2, C3.2, C4.2, U2.3 (VCC)
- new net CAN_Rx: U2.4 (R)
- new net CAN_Tx: U2.1 (D)
Other:
- sheet Monitors renamed Monitor
- sheet Monitor ports: added CRITICAL, PV, SCL, SDA, TC, WARNING; removed none
- sheet Regulators ports: added none; removed +3V3_Sense, +5V_Sense
- moved on the sheet: J1, U1

Commit message: atualização pcb
Parts:
- removed U2: SN65HVD230, Package_SO:SOIC-8_3.9x4.9mm_P1.27mm, symbol Interface_CAN_LIN:SN65HVD230
- added C1: 100nF, Capacitor_SMD:C_0402_1005Metric_Pad0.74x0.62mm_HandSolder, symbol Device:C_Small
- added C7, C9: 33p, symbol Device:C_Small
- added C8: 4n7, symbol Device:C_Small
- added J1: BatBus, Connector_PinHeader_2.54mm:PinHeader_2x06_P2.54mm_Vertical, symbol Connector_Generic:Conn_02x06_Odd_Even
- added R1, R2: 10k, Resistor_SMD:R_0402_1005Metric_Pad0.72x0.64mm_HandSolder, symbol Device:R_Small
- added R3, R4: 4k7, Resistor_SMD:R_0402_1005Metric_Pad0.72x0.64mm_HandSolder, symbol Device:R_Small
- added R5, R6: 60, symbol Device:R_Small
- added U2: SN65HVD233, Package_SO:SOIC-8_3.9x4.9mm_P1.27mm, symbol Interface_CAN_LIN:SN65HVD233
- renumbered C1 to C2, C2 to C3, C3 to C4, C4 to C5, C26 to C6, J1 to J2
Connections:
- net BUS_SCL is gone; now on net BUS_I2C_SCL: J2.19 (Pin_19)
- net BUS_SDA is gone; now on net BUS_I2C_SDA: J2.17 (Pin_17)
- net SOL- is gone; now on net GND: J2.8 (Pin_8)
- net +3.3VP: now also C1.2, J1.7 (Pin_7), J1.8 (Pin_8), R1.1, R2.1, R3.1, R4.1, U2.3 (VCC)
- net +BATT: now also J1.1 (Pin_1), J1.2 (Pin_2)
- net BUS_CAN_H: now also C7.2, R5.1, U2.7 (CANH)
- net BUS_CAN_L: now also C9.1, R6.2, U2.6 (CANL)
- net CAN_Rx: now also U1.44 (PA11), U2.4 (R)
- net CAN_Tx: now also U1.45 (PA12), U2.1 (D)
- net GND: now also C1.1, C7.1, C8.2, C9.2, J1.10 (Pin_10), J1.11 (Pin_11), J1.12 (Pin_12), U2.2 (GND), U2.8 (Rs)
- net UART_Tx: now reaches U1.14 (PA0)
- net UART_Rx: now reaches U1.15 (PA1)
- net I2C2_SCL: now reaches U1.29 (PB10)
- net I2C2_SCL: now also J1.5 (Pin_5), R3.2
- net I2C2_SDA: now reaches U1.30 (PB11)
- net I2C2_SDA: now also J1.6 (Pin_6), R4.2
- net LBK: now reaches U1.38 (PC7)
- net LBK: now also U2.5 (LBK)
- net BUS_I2C_SCL: now reaches U1.58 (PB6)
- net BUS_I2C_SCL: now also R1.2
- net BUS_I2C_SDA: now reaches U1.59 (PB7)
- net BUS_I2C_SDA: now also R2.2
- net BOOT0: now reaches U1.60 (BOOT0)
- net NRST: now reaches U1.7 (NRST)
- new net: C8.1, R5.2, R6.1
- new net Deploy: J1.4 (Pin_4)
- new net Heater: J1.3 (Pin_3)
- new net NTC: J1.9 (Pin_9)
Other:
- moved on the sheet: C2, C3, C4, C5, C6, J2, U1

Commit message: atualização esquema e pcb
Parts:
- added 16M1: Crystal_GND24, Crystal:Crystal_SMD_5032-4Pin_5.0x3.2mm, symbol archive:Device_Crystal_GND24
- added C10, C11: 7p, Capacitor_SMD:C_0402_1005Metric_Pad0.74x0.62mm_HandSolder, symbol archive:Device_C_Small
- added C7: 1u, Capacitor_SMD:C_0402_1005Metric_Pad0.74x0.62mm_HandSolder, symbol archive:Device_C_Small
- added C8, C9: 24p, Capacitor_SMD:C_0402_1005Metric_Pad0.74x0.62mm_HandSolder, symbol archive:Device_C_Small
- added J3: Programmer, Connector_PinHeader_2.54mm:PinHeader_1x12_P2.54mm_Horizontal, symbol archive:Connector_Conn_01x12_Male
- added JP1: BOOT, Jumper:SolderJumper-3_P1.3mm_Open_RoundedPad1.0x1.5mm_NumberLabels, symbol archive:Jumper_SolderJumper_3_Open
- added R1, R2: 10k, Resistor_SMD:R_0402_1005Metric_Pad0.72x0.64mm_HandSolder, symbol archive:Device_R_Small
- added R3: 390, Resistor_SMD:R_0402_1005Metric_Pad0.72x0.64mm_HandSolder, symbol archive:Device_R_Small
- added S1: RST, Button_Switch_SMD:SW_Push_1P1T_NO_CK_KMR2, symbol archive:SamacSys_Parts_PTS636_SM43J_SMTR_LFS
- added Y1: 32,768k, Crystal:Crystal_SMD_3215-2Pin_3.2x1.5mm, symbol archive:Device_Crystal_Small
- C12: renamed from C7; footprint (none) -> Capacitor_SMD:C_0402_1005Metric_Pad0.74x0.62mm_HandSolder
- C13: renamed from C8; footprint (none) -> Capacitor_SMD:C_0402_1005Metric_Pad0.74x0.62mm_HandSolder
- C14: renamed from C9; footprint (none) -> Capacitor_SMD:C_0402_1005Metric_Pad0.74x0.62mm_HandSolder
- R8: renamed from R5; footprint (none) -> Resistor_SMD:R_0603_1608Metric_Pad0.98x0.95mm_HandSolder
- R9: renamed from R6; footprint (none) -> Resistor_SMD:R_0603_1608Metric_Pad0.98x0.95mm_HandSolder
- renumbered R1 to R4, R2 to R5, R3 to R6, R4 to R7
Connections:
- net +3.3V: now also J3.1 (Pin_1), JP1.3 (B), R1.1
- net BOOT0: now also J3.8 (Pin_8), R2.1
- net GND: now also 16M1.2, 16M1.4, C10.2, C11.1, C7.2, C8.2, C9.1, J3.2 (Pin_2), JP1.1 (A), S1.2
- net NRST: now also C7.1, J3.7 (Pin_7), R1.2, S1.1
- net UART_Rx: now also J3.3 (Pin_3)
- net UART_Tx: now also J3.4 (Pin_4)
- net SPI1_SCK: now reaches U1.21 (PA5)
- net SPI1_MISO: now reaches U1.22 (PA6)
- net SPI1_MOSI: now reaches U1.23 (PA7)
- net OSC32_IN: now reaches U1.3 (PC14)
- net OSC32_IN: now also C10.1, Y1.2
- net OSC32_OUT: now reaches U1.4 (PC15)
- net OSC32_OUT: now also C11.2, Y1.1
- net SWDIO: now reaches U1.46 (PA13)
- net SWDIO: now also J3.6 (Pin_6)
- net SWCLK: now reaches U1.49 (PA14)
- net SWCLK: now also J3.5 (Pin_5)
- net OSC_IN: now reaches U1.5 (PH0)
- net OSC_IN: now also 16M1.1, C8.1
- net SWO: now reaches U1.55 (PB3)
- net SWO: now also J3.10 (Pin_10)
- net OSC_OUT: now reaches U1.6 (PH1)
- net OSC_OUT: now also R3.1
- net BUS_MISO: no longer names the net of J2.13 (Pin_13)
- net BUS_MOSI: no longer names the net of J2.14 (Pin_14)
- net BUS_SCLK: no longer names the net of J2.15 (Pin_15)
- net SOL+ renamed SOL_Sense-
- new net: 16M1.3, C9.2, R3.2
- new net: JP1.2 (C), R2.2
- no-connect marks 21 -> 27
Other:
- sheet Charger ports: added none; removed SOL1, SOL2, SOL3, SOL4
- moved on the sheet: C12, C13, C14, J1, R8, R9, U1, U2

Commit message: atualização
Parts:
- removed 16M1: Crystal_GND24, Crystal:Crystal_SMD_5032-4Pin_5.0x3.2mm, symbol archive:Device_Crystal_GND24
- removed C8, C9: 24p, Capacitor_SMD:C_0402_1005Metric_Pad0.74x0.62mm_HandSolder, symbol archive:Device_C_Small
- removed R3: 390, Resistor_SMD:R_0402_1005Metric_Pad0.72x0.64mm_HandSolder, symbol archive:Device_R_Small
- J3: footprint Connector_PinHeader_2.54mm:PinHeader_1x12_P2.54mm_Horizontal -> Connector_Hirose:Hirose_DF13-12P-1.25DSA_1x12_P1.25mm_Vertical
Connections:
- net +3.3V: no longer J3.1 (Pin_1), JP1.3 (B), R1.1
- net +3.3VP: now also J3.1 (Pin_1), JP1.3 (B), R1.1
- net BUS_CAN_H renamed BUS_CAN+
- net BUS_CAN_L renamed BUS_CAN-
- net OSC_IN: no longer names the net of U1.5 (PH0)
- net OSC_OUT: no longer names the net of U1.6 (PH1)
- net SOL_Sense- renamed SOL_Sense+
- no-connect marks 27 -> 29
Other:
- moved on the sheet: C10, C11, Y1

Commit message: atualização pcb/esquema
Parts:
- added D7, D8: LED, LED_SMD:LED_0805_2012Metric_Pad1.15x1.40mm_HandSolder, symbol Device:LED
- added R10, R48: 10k, Resistor_SMD:R_0402_1005Metric_Pad0.72x0.64mm_HandSolder, symbol Device:R_Small
Connections:
- net +3.3VP: now also R10.1, R48.1
- net +3V3_En: now also U1.20 (PA4)
- net +3V3_PG: now also U1.17 (PA3), D7.1 (K)
- net +5V_En: now also U1.37 (PC6)
- net +5V_PG: now also U1.36 (PB15), D8.1 (K)
- net PV: now reaches U1.25 (PC5)
- net CRITICAL: now reaches U1.26 (PB0)
- net WARNING: now reaches U1.27 (PB1)
- net TC: now reaches U1.28 (PB2)
- net ~{CHRG}: now reaches U1.50 (PA15)
- net ~{CHRG}: now also R10.2
- net ~{FAULT}: now reaches U1.51 (PC10)
- net ~{FAULT}: now also R48.2
- net ~{SHDN}: now reaches U1.52 (PC11)
Other:
- sheet Charger ports: added ~{SHDN}; removed none
- moved on the sheet: R5, R6, R7

Commit message: Main Board V1.0
Conclusão da Main Board.
Parts:
- removed J3: Programmer, Connector_Hirose:Hirose_DF13-12P-1.25DSA_1x12_P1.25mm_Vertical, symbol archive:Connector_Conn_01x12_Male
- added D9: LEDR, LED_SMD:LED_0805_2012Metric_Pad1.15x1.40mm_HandSolder, symbol Device:LED
- added J3: Programmer, Connector_Molex:Molex_PicoBlade_53261-1071_1x10-1MP_P1.25mm_Horizontal, symbol Connector:Conn_01x10_Pin
- added J8: External Power, Connector_Molex:Molex_PicoBlade_53261-0671_1x06-1MP_P1.25mm_Horizontal, symbol Connector:Conn_01x06_Socket
- added R49, R50: 470R, Resistor_SMD:R_0402_1005Metric_Pad0.72x0.64mm_HandSolder, symbol Device:R_Small
- added R51: 10k, Resistor_SMD:R_0402_1005Metric_Pad0.72x0.64mm_HandSolder, symbol Device:R_Small
- D7, D8: value LED -> LEDG
Connections:
- net +3.3VP: now also U1.1 (VBAT), J3.1 (Pin_1), R49.1, R50.1
- net +BATT: now also J8.1 (Pin_1), J8.2 (Pin_2)
- net BOOT0: now also J3.8 (Pin_8)
- net Deploy: now also U1.35 (PB14)
- net GND: now also D9.1 (K), J3.2 (Pin_2), J8.5 (Pin_5), J8.6 (Pin_6)
- net Heater: now also U1.34 (PB13)
- net NRST: now also J3.7 (Pin_7)
- net SPI1_MISO: now also J2.13 (Pin_13)
- net SPI1_MOSI: now also J2.14 (Pin_14)
- net SPI1_SCK: now also J2.15 (Pin_15)
- net SWCLK: now also J3.5 (Pin_5)
- net SWDIO: now also J3.6 (Pin_6)
- net SWO: now also J3.10 (Pin_10)
- net UART_Rx: now also J3.3 (Pin_3)
- net UART_Tx: now also J3.4 (Pin_4)
- net at D8.2 (A): now also R50.2
- net DebugLed: now reaches U1.9 (PC1)
- net DebugLed: now also R51.1
- net at D7.2 (A): now also R49.2
- net SOL_Sense+ renamed SOL+
- net SOL+: now also J8.4 (Pin_4)
- new net: D9.2 (A), R51.2
- no-connect marks 29 -> 43
Other:
- note removed: "Cuidado para não inverter o lado da pcb"
- moved on the sheet: D7
