File: Main Board/Kicad/monitors.kicad_sch (KiCad schematic)
At the start: 3 parts, among them U5 INA3221, U6 INA3221, U7 INA3221

Commit message: Atualização do circuito/pcb
Parts:
- renumbered U7 to U5, U5 to U6, U6 to U7
Changed lines of the file:
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@@
 		(dnp no)
 		(fields_autoplaced yes)
-		(property "Reference" "U6"
+		(property "Reference" "U7"
 			(at 150.7333 99.06 0)
 			(show_name no)
@@
 			(project "Power Supply ZensatV3"
 				(path "/64de738a-78a3-405a-9208-2090dc1f201b/87265ed7-3614-439d-98ab-bc8ca0914738"
-					(reference "U6")
+					(reference "U7")
 					(unit 1)
 				)
@@
 		(dnp no)
 		(fields_autoplaced yes)
-		(property "Reference" "U7"
+		(property "Reference" "U5"
 			(at 205.3433 50.8 0)
 			(show_name no)
@@
 			(project "Power Supply ZensatV3"
 				(path "/64de738a-78a3-405a-9208-2090dc1f201b/87265ed7-3614-439d-98ab-bc8ca0914738"
-					(reference "U7")
+					(reference "U5")
 					(unit 1)
 				)
@@
 		(dnp no)
 		(fields_autoplaced yes)
-		(property "Reference" "U5"
+		(property "Reference" "U6"
 			(at 150.7333 52.07 0)
 			(show_name no)
@@
 			(project "Power Supply ZensatV3"
 				(path "/64de738a-78a3-405a-9208-2090dc1f201b/87265ed7-3614-439d-98ab-bc8ca0914738"
-					(reference "U5")
+					(reference "U6")
 					(unit 1)
 				)
@@
 		(dnp no)
 		(fields_autoplaced yes)
-		(property "Reference" "#PWR05"
+		(property "Reference" "#PWR015"
 			(at 143.51 96.52 0)
 			(hide yes)
@@
 			(project "Power Supply ZensatV3"
 				(path "/64de738a-78a3-405a-9208-2090dc1f201b/87265ed7-3614-439d-98ab-bc8ca0914738"
-					(reference "#PWR05")
+					(reference "#PWR015")
 					(unit 1)
 				)
@@
 		(dnp no)
 		(fields_autoplaced yes)
-		(property "Reference" "#PWR07"
+		(property "Reference" "#PWR014"
 			(at 198.12 95.25 0)
 			(hide yes)
@@
 			(project "Power Supply ZensatV3"
 				(path "/64de738a-78a3-405a-9208-2090dc1f201b/87265ed7-3614-439d-98ab-bc8ca0914738"
-					(reference "#PWR07")
+					(reference "#PWR014")
 					(unit 1)
 				)
@@
 		(dnp no)
 		(fields_autoplaced yes)
-		(property "Reference" "#PWR06"
+		(property "Reference" "#PWR016"
 			(at 143.51 143.51 0)
 			(hide yes)
@@
 			(project "Power Supply ZensatV3"
 				(path "/64de738a-78a3-405a-9208-2090dc1f201b/87265ed7-3614-439d-98ab-bc8ca0914738"
-					(reference "#PWR06")
+					(reference "#PWR016")
 					(unit 1)
 				)

Commit message: atualização pcb
Parts:
- removed U5, U7: INA3221, Package_DFN_QFN:Texas_RGV0016A_VQFN-16-1EP_4x4mm_P0.65mm_EP2.1x2.1mm, symbol Power_Management:INA3221
- added C21: 100nF, Capacitor_SMD:C_0402_1005Metric_Pad0.74x0.62mm_HandSolder, symbol Device:C_Small
- added JP1, JP2, JP3, JP4, JP5: SolderJumper_2_Open, Jumper:SolderJumper-2_P1.3mm_Open_RoundedPad1.0x1.5mm, symbol Jumper:SolderJumper_2_Open
- added R10, R7, R8, R9: 10k, Resistor_SMD:R_0402_1005Metric_Pad0.72x0.64mm_HandSolder, symbol Device:R_Small
Connections:
- net GND: now also U6.17 (EP), C21.1, JP5.2 (B)
- net +3.3V: now reaches U6.1 (IN-3)
- net PV: now reaches U6.10 (PV)
- net PV: now also R7.1
- net +5V: now reaches U6.11 (IN-1)
- net +5V_Sense: now reaches U6.12 (IN+1)
- net TC: now reaches U6.13 (TC)
- net TC: now also R10.1
- net -SOL_Sense: now reaches U6.14 (IN-2)
- net +SOL_Sense: now reaches U6.15 (IN+2)
- net at U6.16 (VPU): now also JP1.1 (A), R7.2
- net +3V3_Sense: now reaches U6.2 (IN+3)
- net +3.3VP: now reaches U6.4 (VS)
- net +3.3VP: now also C21.2, JP1.2 (B), JP2.2 (B), R10.2, R8.2, R9.2
- net at U6.5 (A0): now also JP2.1 (A), JP3.1 (A), JP4.1 (A), JP5.1 (A)
- net SCL: now reaches U6.6 (SCL)
- net SCL: now also JP4.2 (B)
- net SDA: now reaches U6.7 (SDA)
- net SDA: now also JP3.2 (B)
- net WARNING: now reaches U6.8 (WARNING)
- net WARNING: now also R9.1
- net CRITICAL: now reaches U6.9 (CRITICAL)
- net CRITICAL: now also R8.1
Other:
- note added: "I/V Monitor"
- moved on the sheet: U6

Commit message: atualização pcb
Parts:
- removed JP2, JP3, JP4, JP5: SolderJumper_2_Open, Jumper:SolderJumper-2_P1.3mm_Open_RoundedPad1.0x1.5mm, symbol Jumper:SolderJumper_2_Open
- added C27, C28, C29, C30: 100nF, Capacitor_SMD:C_0402_1005Metric_Pad0.74x0.62mm_HandSolder, symbol Device:C_Small
- added R15, R16, R21, R22, R24, R27: 10R, Resistor_SMD:R_0402_1005Metric_Pad0.72x0.64mm_HandSolder, symbol Device:R_Small
- added R23, R25, R26, R28: 0R, Resistor_SMD:R_0402_1005Metric_Pad0.72x0.64mm_HandSolder, symbol Device:R_Small
- added U6: LM75B, Package_SO:VSSOP-8_3x3mm_P0.65mm, symbol Sensor_Temperature:LM75B
- renumbered C21 to C26, R7 to R17, R8 to R18, R9 to R19, R10 to R20, U6 to U7
Connections:
- net +3.3V: now also R27.2; no longer U7.1 (IN-3)
- net +3.3VP: now also C28.2, R23.1, U6.8 (+Vs)
- net +3V3_Sense: now also R24.2; no longer U7.2 (IN+3)
- net +5V: now also R16.2; no longer U7.11 (IN-1)
- net +5V_Sense: now also R15.2; no longer U7.12 (IN+1)
- net GND: now also C28.1, R28.1, U6.4 (GND), U6.5 (A2), U6.6 (A1), U6.7 (A0)
- net SCL: now also R26.1, U6.2 (SCL)
- net SDA: now also R25.1, U6.1 (SDA)
- net at U7.5 (A0): now also R23.2, R25.2, R26.2, R28.2
- net +SOL_Sense: no longer names the net of U7.15 (IN+2)
- net +SOL_Sense: now also C29.1, R21.1
- net -SOL_Sense: no longer names the net of U7.14 (IN-2)
- net -SOL_Sense: now also C29.2, R22.1
- new net: C27.1, R15.1, U7.12 (IN+1)
- new net: C30.2, R27.1, U7.1 (IN-3)
- new net: C27.2, R16.1, U7.11 (IN-1)
- new net: C30.1, R24.1, U7.2 (IN+3)
- new net SOL_Sense+: R21.2
- new net SOL_Sense-: R22.2
- no-connect marks 0 -> 1
Other:
- note added: "Resistores para escolha do endereço. Usar apenas 1."

Commit message: atualização esquema e pcb
Parts:
- added R26, R28, R31, R34: 0R, Resistor_SMD:R_0402_1005Metric_Pad0.72x0.64mm_HandSolder, symbol Device:R_Small
- U6: footprint Package_SO:VSSOP-8_3x3mm_P0.65mm -> Package_SO:Texas_S-PDSO-G8_3x3mm_P0.65mm
- renumbered C26 to C31, C27 to C32, C28 to C33, C29 to C34, C30 to C35, JP1 to JP2, R15 to R20, R16 to R21, R17 to R22, R18 to R23, R19 to R24, R20 to R25, R21 to R27, R22 to R29, R23 to R30, R24 to R32, R25 to R33, R26 to R35, R27 to R36, R28 to R37
Connections:
- net +3.3VP: now also R26.1, R31.1
- net GND: now also R28.1, R34.1; no longer U6.6 (A1), U6.7 (A0)
- new net: R31.2, R34.2, U6.6 (A1)
- new net: R26.2, R28.2, U6.7 (A0)
Other:
- moved on the sheet: C31, C32, C33, C34, C35, JP2, R20, R21, R22, R23, R24, R25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

Commit message: atualização
Parts:
- removed JP2: SolderJumper_2_Open, Jumper:SolderJumper-2_P1.3mm_Open_RoundedPad1.0x1.5mm, symbol Jumper:SolderJumper_2_Open
Connections:
- net +3.3VP: now also R22.2, U7.16 (VPU)
Changed lines of the file:
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@@
 	(wire
 		(pts
-			(xy 191.77 71.12) (xy 196.85 71.12)
-		)
-		(stroke
-			(width 0)
-			(type default)
-		)
-	)
-	(wire
-		(pts
 			(xy 67.31 78.74) (xy 67.31 88.9)
 		)
@@
 	(wire
 		(pts
-			(xy 180.34 71.12) (xy 181.61 71.12)
-		)
-		(stroke
-			(width 0)
-			(type default)
-		)
-	)
-	(wire
-		(pts
 			(xy 196.85 71.12) (xy 196.85 74.93)
 		)
@@
 	(wire
 		(pts
+			(xy 180.34 71.12) (xy 196.85 71.12)
+		)
+		(stroke
+			(width 0)
+			(type default)
+		)
+	)
+	(wire
+		(pts
 			(xy 34.29 87.63) (xy 31.75 87.63)
 		)
@@
 					(unit 1)
 				)
-			)
-		)
-	)
-	(symbol
-		(lib_id "Jumper:SolderJumper_2_Open")
-		(at 186.69 71.12 180)
-		(unit 1)
-		(body_style 1)
-		(exclude_from_sim no)
-		(in_bom no)
-		(on_board yes)
-		(in_pos_files yes)
-		(dnp no)
-		(property "Reference" "JP2"
-			(at 186.69 73.914 0)
-			(show_name no)
-			(do_not_autoplace no)
-			(effects
-				(font
-					(size 1.27 1.27)
-				)
-			)
-		)
-		(property "Value" "SolderJumper_2_Open"
-			(at 186.69 74.93 0)
-			(hide yes)
-			(show_name no)
-			(do_not_autoplace no)
-			(effects
-				(font
-					(size 1.27 1.27)
-				)
-			)
-		)
-		(property "Footprint" "Jumper:SolderJumper-2_P1.3mm_Open_RoundedPad1.0x1.5mm"
-			(at 186.69 71.12 0)
-			(hide yes)
-			(show_name no)
-			(do_not_autoplace no)
-			(effects
-				(font
-					(size 1.27 1.27)
-				)
-			)
-		)
-		(property "Datasheet" ""
-			(at 186.69 63.5 0)
-			(hide yes)
-			(show_name no)
-			(do_not_autoplace no)
-			(effects
-				(font
-					(size 1.27 1.27)
-				)
-			)
-		)
-		(property "Description" "Solder Jumper, 2-pole, open"
-			(at 186.69 66.04 0)
-			(hide yes)
-			(show_name no)
-			(do_not_autoplace no)
-			(effects
-				(font
-					(size 1.27 1.27)
-				)
-			)
-		)
-		(pin "1"
-		)
-		(pin "2"
-		)
-		(instances
-			(project "Power Supply ZensatV3"
-				(path "/64de738a-78a3-405a-9208-2090dc1f201b/87265ed7-3614-439d-98ab-bc8ca0914738"
-					(reference "JP2")
-					(unit 1)
-				)

Commit message: atualização pcb/esquema
Parts:
- C31, C32, C34, C35: value 100nF -> 100nF 10V
Changed lines of the file:
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@@
 			)
 		)
-		(property "Value" "100nF"
+		(property "Value" "100nF 10V"
 			(at 138.43 116.8462 0)
 			(show_name no)
@@
 			)
 		)
-		(property "Value" "100nF"
+		(property "Value" "100nF 10V"
 			(at 138.43 95.2562 0)
 			(show_name no)
@@
 			)
 		)
-		(property "Value" "100nF"
+		(property "Value" "100nF 10V"
 			(at 186.6836 58.42 90)
 			(show_name no)
@@
 			)
 		)
-		(property "Value" "100nF"
+		(property "Value" "100nF 10V"
 			(at 138.43 73.6662 0)
 			(show_name no)

Commit message: Main Board V1.0
Conclusão da Main Board.
Connections:
- net SOL_Sense+ renamed SOL+
Changed lines of the file:
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@@
-		)
-	)
-	(text "Resistores para escolha do endereço.\nUsar apenas 1."
-		(exclude_from_sim no)
-		(at 58.42 132.588 0)
-		(effects
-			(font
-				(size 1.27 1.27)
-			)
 		)
 	)
@@
 		)
 	)
-	(global_label "SOL_Sense+"
+	(global_label "SOL+"
 		(shape input)
 		(at 124.46 88.9 180)
@@
 		)
 		(property "Intersheetrefs" "${INTERSHEET_REFS}"
-			(at 109.8029 88.9 0)
+			(at 116.3343 88.9 0)
 			(hide yes)
 			(show_name no)
