File: Main Board/Kicad/regulators.kicad_sch (KiCad schematic)
At the start: 27 parts, among them U2 LMR33630ADDA, U3 LMR33630ADDA, U4 AMS1117-3.3

Commit message: Atualização do circuito/pcb
Parts:
- R1: renamed from R5; footprint (none) -> Resistor_SMD:R_0612_1632Metric_Pad1.18x3.40mm_HandSolder
- R4: renamed from R6; footprint (none) -> Resistor_SMD:R_0612_1632Metric_Pad1.18x3.40mm_HandSolder
- renumbered C6 to C1, C12 to C11, C14 to C12, C16 to C13, C4 to C14, C5 to C15, C8 to C16, C1 to C2, C9 to C3, C11 to C4, C13 to C5, C15 to C6, C3 to C7, C7 to C8, C2 to C9, R1 to R2, R2 to R3, R3 to R5, R4 to R6

Commit message: atualização pcb
Parts:
- C11: renamed from C7; footprint Capacitor_SMD:C_0402_1005Metric_Pad0.74x0.62mm_HandSolder -> Capacitor_SMD:C_0603_1608Metric_Pad1.08x0.95mm_HandSolder
- C13: renamed from C9; footprint Capacitor_SMD:C_1206_3216Metric_Pad1.33x1.80mm_HandSolder -> Capacitor_SMD:C_0805_2012Metric_Pad1.18x1.45mm_HandSolder
- C18: renamed from C14; footprint Capacitor_SMD:C_0402_1005Metric_Pad0.74x0.62mm_HandSolder -> Capacitor_SMD:C_0603_1608Metric_Pad1.08x0.95mm_HandSolder
- C20: renamed from C16; footprint Capacitor_SMD:C_1206_3216Metric_Pad1.33x1.80mm_HandSolder -> Capacitor_SMD:C_0805_2012Metric_Pad1.18x1.45mm_HandSolder
- C6: renamed from C2; footprint Capacitor_SMD:C_1206_3216Metric_Pad1.33x1.80mm_HandSolder -> Capacitor_SMD:C_0805_2012Metric_Pad1.18x1.45mm_HandSolder
- renumbered C6 to C10, C8 to C12, C10 to C14, C11 to C15, C12 to C16, C13 to C17, C15 to C19, C1 to C5, C3 to C7, C4 to C8, C5 to C9, U2 to U3, U3 to U4, U4 to U5
Connections:
- net BATC+ is gone; now on net +BATT: C19.2, U5.3 (VI)
Other:
- moved on the sheet: C10, C11, C19, C20, C5, C6, C7, C8, C9, L1, R1, R2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

Commit message: atualização pcb
Parts:
- added R11, R7: *0R, Resistor_SMD:R_0402_1005Metric_Pad0.72x0.64mm_HandSolder, symbol Device:R_Small
- renumbered C5 to C10, C6 to C11, C7 to C12, C8 to C13, C9 to C14, C10 to C15, C11 to C16, C12 to C17, C13 to C18, C14 to C19, C15 to C20, C16 to C21, C17 to C22, C18 to C23, C19 to C24, C20 to C25, R3 to R10, R4 to R12, R5 to R13, R6 to R14, R1 to R8, R2 to R9
Connections:
- net +3V3_Enable: now also R7.2
- net +5V_Enable: now also R11.2
- net +BATT: now also R11.1, R7.1
Other:
- note added: "*Usar para o modo de operação sem o microcontrolador"
- moved on the sheet: C11, C18

Commit message: atualização esquema e pcb
Parts:
- added R14, R19: 10k, Resistor_SMD:R_0402_1005Metric_Pad0.72x0.64mm_HandSolder, symbol Device:R_Small
- renumbered C10 to C15, C11 to C16, C12 to C17, C13 to C18, C14 to C19, C15 to C20, C16 to C21, C17 to C22, C18 to C23, C19 to C24, C20 to C25, C21 to C26, C22 to C27, C23 to C28, C24 to C29, C25 to C30, R7 to R10, R8 to R11, R9 to R12, R10 to R13, R11 to R15, R12 to R16, R13 to R17, R14 to R18
Connections:
- net +3.3VP: now also R14.1, R19.1
- net +3V3_PG: now also R14.2
- net +5V_PG: now also R19.2

Commit message: atualização
Parts:
- removed R10, R15: *0R, Resistor_SMD:R_0402_1005Metric_Pad0.72x0.64mm_HandSolder, symbol Device:R_Small
Changed lines of the file:
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@@
 	)
 	(junction
-		(at 107.95 43.18)
-		(diameter 0)
-		(color 0 0 0 0)
-	)
-	(junction
 		(at 180.34 60.96)
 		(diameter 0)
@@
 	)
 	(junction
-		(at 107.95 88.9)
-		(diameter 0)
-		(color 0 0 0 0)
-	)
-	(junction
 		(at 82.55 88.9)
 		(diameter 0)
@@
 	)
 	(junction
-		(at 107.95 48.26)
-		(diameter 0)
-		(color 0 0 0 0)
-	)
-	(junction
 		(at 139.7 140.97)
 		(diameter 0)
@@
 	)
 	(junction
-		(at 107.95 93.98)
-		(diameter 0)
-		(color 0 0 0 0)
-	)
-	(junction
 		(at 190.5 45.72)
 		(diameter 0)
@@
 	(wire
 		(pts
-			(xy 82.55 88.9) (xy 107.95 88.9)
-		)
-		(stroke
-			(width 0)
-			(type default)
-		)
-	)
-	(wire
-		(pts
 			(xy 210.82 45.72) (xy 217.17 45.72)
 		)
@@
 	(wire
 		(pts
-			(xy 107.95 88.9) (xy 115.57 88.9)
+			(xy 82.55 88.9) (xy 115.57 88.9)
 		)
 		(stroke
@@
 	(wire
 		(pts
-			(xy 107.95 93.98) (xy 115.57 93.98)
+			(xy 104.14 93.98) (xy 115.57 93.98)
 		)
 		(stroke
@@
 	(wire
 		(pts
-			(xy 104.14 93.98) (xy 107.95 93.98)
-		)
-		(stroke
-			(width 0)
-			(type default)
-		)
-	)
-	(wire
-		(pts
 			(xy 170.18 45.72) (xy 180.34 45.72)
 		)
@@
 	(wire
 		(pts
-			(xy 104.14 48.26) (xy 107.95 48.26)
+			(xy 104.14 48.26) (xy 115.57 48.26)
 		)
 		(stroke
@@
 	(wire
 		(pts
-			(xy 107.95 43.18) (xy 115.57 43.18)
-		)
-		(stroke
-			(width 0)
-			(type default)
-		)
-	)
-	(wire
-		(pts
 			(xy 156.21 97.79) (xy 156.21 99.06)
 		)
@@
 	(wire
 		(pts
-			(xy 82.55 43.18) (xy 107.95 43.18)
+			(xy 82.55 43.18) (xy 115.57 43.18)
 		)
 		(stroke
@@
 	(wire
 		(pts
-			(xy 107.95 48.26) (xy 115.57 48.26)
-		)
-		(stroke
-			(width 0)
-			(type default)
-		)
-	)
-	(wire
-		(pts
 			(xy 170.18 106.68) (xy 156.21 106.68)
 		)
@@
 	)
 	(symbol
-		(lib_id "Device:R_Small")
-		(at 107.95 91.44 0)
-		(unit 1)
-		(body_style 1)
-		(exclude_from_sim no)
-		(in_bom yes)
-		(on_board yes)
-		(in_pos_files yes)
-		(dnp no)
-		(fields_autoplaced yes)
-		(property "Reference" "R15"
-			(at 110.49 90.1699 0)
-			(show_name no)
-			(do_not_autoplace no)
-			(effects
-				(font
-					(size 1.016 1.016)
-				)
-				(justify left)
-			)
-		)
-		(property "Value" "*0R"
-			(at 110.49 92.7099 0)
-			(show_name no)
-			(do_not_autoplace no)
-			(effects
-				(font
-					(size 1.27 1.27)
-				)
-				(justify left)
-			)
-		)
-		(property "Footprint" "Resistor_SMD:R_0402_1005Metric_Pad0.72x0.64mm_HandSolder"
-			(at 107.95 91.44 0)
-			(hide yes)
-			(show_name no)
-			(do_not_autoplace no)
-			(effects
-				(font
-					(size 1.27 1.27)
-				)
-			)
-		)
-		(property "Datasheet" ""
-			(at 107.95 91.44 0)
-			(hide yes)
-			(show_name no)
-			(do_not_autoplace no)
-			(effects
-				(font
-					(size 1.27 1.27)
-				)
-			)
-		)
-		(property "Description" "Resistor, small symbol"
-			(at 107.95 91.44 0)
-			(hide yes)
-			(show_name no)
-			(do_not_autoplace no)
-			(effects
-				(font
-					(size 1.27 1.27)
-				)
-			)
-		)
-		(pin "1"
-		)
-		(pin "2"
-		)
-		(instances
-			(project "Power Supply ZensatV3"
-				(path "/64de738a-78a3-405a-9208-2090dc1f201b/4e272359-939b-4428-bdf1-656f4c28d372"
-					(reference "R15")
-					(unit 1)
-				)
-			)
-		)
-	)
-	(symbol
 		(lib_id "Device:C_Small")
 		(at 82.55 50.8 180)
@@
 					(unit 1)
 				)
-			)
-		)
-	)
-	(symbol
-		(lib_id "Device:R_Small")
-		(at 107.95 45.72 0)
-		(unit 1)
-		(body_style 1)
-		(exclude_from_sim no)
-		(in_bom yes)
-		(on_board yes)
-		(in_pos_files yes)
-		(dnp no)
-		(fields_autoplaced yes)
-		(property "Reference" "R10"
-			(at 110.49 44.4499 0)
-			(show_name no)
-			(do_not_autoplace no)
-			(effects
-				(font
-					(size 1.016 1.016)
-				)
-				(justify left)
-			)
-		)
-		(property "Value" "*0R"
-			(at 110.49 46.9899 0)
-			(show_name no)
-			(do_not_autoplace no)
-			(effects
-				(font
-					(size 1.27 1.27)
-				)
-				(justify left)
-			)
-		)
-		(property "Footprint" "Resistor_SMD:R_0402_1005Metric_Pad0.72x0.64mm_HandSolder"
-			(at 107.95 45.72 0)
-			(hide yes)
-			(show_name no)
-			(do_not_autoplace no)
-			(effects
-				(font
-					(size 1.27 1.27)
-				)
-			)
-		)
-		(property "Datasheet" ""
-			(at 107.95 45.72 0)
-			(hide yes)
-			(show_name no)
-			(do_not_autoplace no)
-			(effects
-				(font
-					(size 1.27 1.27)
-				)
-			)
-		)
-		(property "Description" "Resistor, small symbol"
-			(at 107.95 45.72 0)
-			(hide yes)
-			(show_name no)
-			(do_not_autoplace no)
-			(effects
-				(font
-					(size 1.27 1.27)
-				)
-			)
-		)
-		(pin "1"
-		)
-		(pin "2"
-		)
-		(instances
-			(project "Power Supply ZensatV3"
-				(path "/64de738a-78a3-405a-9208-2090dc1f201b/4e272359-939b-4428-bdf1-656f4c28d372"
-					(reference "R10")
-					(unit 1)
-				)

Commit message: atualização pcb/esquema
Parts:
- added C41, C42: 220nF, Capacitor_SMD:C_0402_1005Metric_Pad0.74x0.62mm_HandSolder, symbol Device:C_Small
- added R15, R47: 1k, Resistor_SMD:R_0402_1005Metric_Pad0.72x0.64mm_HandSolder, symbol Device:R_Small
- C29: value 100nF -> 100nF 25V
- C30: value 10uF -> 10uF 10V
Connections:
- net +3V3_Enable: now also R15.1; no longer U3.3 (EN)
- net +5V_Enable: now also R47.1; no longer U4.3 (EN)
- net +BATT: now also C41.2, C42.2
- net GND: now also C41.1, C42.1
- new net: R15.2, U3.3 (EN)
- new net: R47.2, U4.3 (EN)
Other:
- note added: "25V Capacitors"
- moved on the sheet: C16, C23, C29, C30

Commit message: Main Board V1.0
Conclusão da Main Board.
Other:
- note removed: "*Usar para o modo de operação sem o microcontrolador"
Changed lines of the file:
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@@
-		)
-	)
-	(text "*Usar para o modo de operação sem o microcontrolador"
-		(exclude_from_sim no)
-		(at 211.074 158.242 0)
-		(effects
-			(font
-				(size 1.27 1.27)
-			)
 		)
 	)

Commit message: Finalização V1.5
Parts:
- R18: value 14,9k -> 24,9k
Changed lines of the file:
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@@
 			)
 		)
-		(property "Value" "14,9k"
+		(property "Value" "24,9k"
 			(at 158.75 104.1399 0)
 			(show_name no)
