File: Main Board/Kicad/regulators.kicad_sch (KiCad schematic)
At the start: 33 parts, among them U3 LMR33630ADDA, U4 LMR33630ADDA, U5 AMS1117-3.3

Commit message: Final V1.0
Finalização da primeira versão.
Parts:
- C30: value 10uF 10V -> 10uF 10V Tantalum
Changed lines of the file:
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@@
 			)
 		)
-		(property "Value" "10uF 10V"
+		(property "Value" "10uF 10V Tantalum"
 			(at 147.32 147.3135 0)
 			(show_name no)
